File: Audio.sch (KiCad schematic (older format))
At the start: 53 parts, among them J5 PJ-3270, J6 PJ-3270, J7 PJ-3270, U6 SSM2603, Y1 12.288Mhz

Commit message: OtterCastAmp inital commit
Parts:
- J5, J6, J7: symbol otter:PJ-3270 -> OtterCastAmp-rescue:PJ-3270-otter
- U6: symbol otter:SSM2603 -> OtterCastAmp-rescue:SSM2603-otter
Changed lines of the file:
@@
 BT-PCM-DOUT
 $Comp
-L otter:SSM2603 U6
+L OtterCastAmp-rescue:SSM2603-otter U6
 U 1 1 5FF6F21F
 P 5750 4050
@@
 $EndComp
 $Comp
-L otter:GND #PWR0205
+L OtterCastAmp-rescue:GND-otter #PWR0205
 U 1 1 5FF88FDC
 P 5850 5800
@@
 $EndComp
 $Comp
-L otter:GND #PWR0206
+L OtterCastAmp-rescue:GND-otter #PWR0206
 U 1 1 5FF8C63C
 P 6050 5800
@@
 $EndComp
 $Comp
-L S3-OLinuXino_Rev_A:GND #PWR?
+L OtterCastAmp-rescue:GND-S3-OLinuXino_Rev_A #PWR?
 U 1 1 5FF96B43
 P 4850 5150
@@
 Connection ~ 4750 5250
 $Comp
-L S3-OLinuXino_Rev_A:GND #PWR?
+L OtterCastAmp-rescue:GND-S3-OLinuXino_Rev_A #PWR?
 U 1 1 5FF96B59
 P 4650 5150
@@
 	4750 5250 4400 5250
 $Comp
-L S3-OLinuXino_Rev_A:GND #PWR?
+L OtterCastAmp-rescue:GND-S3-OLinuXino_Rev_A #PWR?
 U 1 1 5FF96B61
 P 4100 5050
@@
 	4100 5050 4200 5050
 $Comp
-L S3-OLinuXino_Rev_A:GND #PWR?
+L OtterCastAmp-rescue:GND-S3-OLinuXino_Rev_A #PWR?
 U 1 1 5FF96B68
 P 4100 5250
@@
 $EndComp
 $Comp
-L S3-OLinuXino_Rev_A:+3.3V #PWR?
+L OtterCastAmp-rescue:+3.3V-S3-OLinuXino_Rev_A #PWR?
 U 1 1 5FFB96F5
 P 4100 4550
@@
 Connection ~ 6750 2100
 $Comp
-L otter:GND #PWR0213
+L OtterCastAmp-rescue:GND-otter #PWR0213
 U 1 1 601BC91C
 P 6800 2400
@@
 Connection ~ 6750 2400
 $Comp
-L otter:GND #PWR0214
+L OtterCastAmp-rescue:GND-otter #PWR0214
 U 1 1 601C6C24
 P 6600 2000
@@
 	4850 1700 5150 1700
 $Comp
-L S3-OLinuXino_Rev_A:+3.0VA #PWR?
+L OtterCastAmp-rescue:+3.0VA-S3-OLinuXino_Rev_A #PWR?
 U 1 1 6023A1C9
 P 6600 1700
@@
 Connection ~ 4850 1700
 $Comp
-L S3-OLinuXino_Rev_A:+3.0VA #PWR?
+L OtterCastAmp-rescue:+3.0VA-S3-OLinuXino_Rev_A #PWR?
 U 1 1 6027AD71
 P 4250 1700
@@
 $EndComp
 $Comp
-L S3-OLinuXino_Rev_A:+3.0VA #PWR?
+L OtterCastAmp-rescue:+3.0VA-S3-OLinuXino_Rev_A #PWR?
 U 1 1 602F2215
 P 4250 2100
@@
 	6750 5400 6750 5350
 $Comp
-L otter:GND #PWR0231
+L OtterCastAmp-rescue:GND-otter #PWR0231
 U 1 1 60A50D39
 P 6800 5400
@@
 Connection ~ 6400 5100
 $Comp
-L otter:PJ-3270 J7
+L OtterCastAmp-rescue:PJ-3270-otter J7
 U 1 1 60B772BD
 P 9050 2900
@@
 $EndComp
 $Comp
-L otter:PJ-3270 J6
+L OtterCastAmp-rescue:PJ-3270-otter J6
 U 1 1 60B798B5
 P 8450 3400
@@
 $EndComp
 $Comp
-L otter:PJ-3270 J5
+L OtterCastAmp-rescue:PJ-3270-otter J5
 U 1 1 60B92BDF
 P 3200 3100
@@
 	2950 2500 2950 2450
 $Comp
-L S3-OLinuXino_Rev_A:+3.0VA #PWR?
+L OtterCastAmp-rescue:+3.0VA-S3-OLinuXino_Rev_A #PWR?
 U 1 1 60C3B44B
 P 2950 2200
@@
 $EndComp
 $Comp
-L otter:GND #PWR0295
+L OtterCastAmp-rescue:GND-otter #PWR0295
 U 1 1 5FE5C65A
 P 5850 6600

Commit message: started layout
Parts:
- removed C54, C55, C56, C57, C60, C62, C63, C64, C69: 10u, otter:CP_EIA-3216-10, symbol Device:CP_Small
- removed C58, C59: 100n, otter:C_0402, symbol Device:C_Small
- removed C67, C68: 100u, otter:CP_EIA-3528-12, symbol Device:CP_Small
- removed FB2, FB3: FERRET, otter:R_0805, symbol Device:Ferrite_Bead_Small
- removed J5, J6, J7: PJ-3270, otter:PJ-3270, symbol OtterCastAmp-rescue:PJ-3270-otter
- removed MK1: Mic, otter:B4013AM422-42, symbol Device:Microphone
- removed R27: 0R, otter:R_0805, symbol Device:R_Small
- removed R47, R52: DNP, otter:R_0402, symbol Device:R_Small
- removed R48, R49, R50, R51: 2k2, otter:R_0402, symbol Device:R_Small
- removed R54: 22, otter:R_0402, symbol Device:R_Small
- removed R58, R59, R60, R63: 47k, otter:R_0402, symbol Device:R_Small
- removed R61, R62: 100, otter:R_0402, symbol Device:R_Small
- removed U6: SSM2603, otter:LFCSP-28-5x5mm-0.5mm-EP3.14x3.14mm, symbol OtterCastAmp-rescue:SSM2603-otter
- removed Y1: 12.288Mhz, otter:Oscillator_3225, symbol Device:Crystal_GND24_Small
- added C43, C62: 100n, otter:C_0402, symbol Device:C_Small
- added C44, C63: 10u, otter:C_0603, symbol Device:C_Small
- added C45, C64: 1u, otter:C_0402, symbol Device:C_Small
- added C48, C49, C67, C68: 100n 50V, otter:C_0603, symbol Device:C_Small
- added C54, C55, C73, C74: 22u 50V, Capacitor_SMD:C_1206_3216Metric, symbol Device:C_Small
- added C56, C60, C69, C75, C79: 470n 25V, otter:C_0603, symbol Device:C_Small
- added C57, C72, C76, C80: 680n 50V, Capacitor_SMD:C_1206_3216Metric, symbol Device:C_Small
- added C58, C59, C77, C78: 470u 35V, Capacitor_SMD:CP_Elec_10x10.5, symbol Device:CP_Small
- added H1, H2: 3.2mm, MountingHole:MountingHole_3.2mm_M3_Pad_Via, symbol Mechanical:MountingHole_Pad
- added J5, J6: C475204, otter:C475204, symbol Connector_Generic:Conn_01x04
- added JP1, JP2, JP3, JP4, JP5, JP6, JP7, JP8: PBTL, Jumper:SolderJumper-2_P1.3mm_Open_Pad1.0x1.5mm, symbol Device:Jumper_NC_Small
- added L10, L11, L4, L5, L6, L7, L8, L9: 10u, otter:L_10.4x10.4_H4.8, symbol Device:L_Small
- added R37, R38, R39: 10k, otter:R_0402, symbol Device:R_Small
- added U10, U9: TAS5825MRHB, Package_DFN_QFN:Texas_S-PVQFN-N32_EP3.45x3.45mm, symbol Amplifier_Audio:TAS5825MRHB
- C46: value 220p -> 1u
- C47: value 1n -> 1u
- C50, C71: value 220p -> 470n 25V; footprint otter:C_0402 -> otter:C_0603
- C51: value 18p -> 680n 50V; footprint otter:C_0402 -> Capacitor_SMD:C_1206_3216Metric
- C52: value 18p -> 470n 25V; footprint otter:C_0402 -> otter:C_0603
- C53, C70: value 220p -> 680n 50V; footprint otter:C_0402 -> Capacitor_SMD:C_1206_3216Metric
- C61: value 100n -> 680n 50V; footprint otter:C_0402 -> Capacitor_SMD:C_1206_3216Metric
- C65, C66: value 100n -> 1u
- R40: value 200k -> 0R
- R41: value 2k2 -> 0R
- R42: value 47k -> 10k
- R43: value 680 -> 10k
- R44: value 0 -> 10k
- R45: value 0 -> DNP
- R46: value 0 -> 1k
Connections:
- net +3V3: now also R42.1, R43.1, R44.1, R37.1, R38.1, R39.1; no longer C66.1
- net GND: now also C46.1, C47.1, C51.1, C53.2, C65.1, C66.1, C70.1, R40.2, R46.2, C43.1, C44.1, C45.1, C48.2, C49.2, C54.2, C55.2, C57.1, C58.2, C59.2, C62.1, C63.1, C64.1, C67.2, C68.2, C72.2, C73.2, C74.2, C76.1, C77.2, C78.2, C80.2, H1.1, H2.1, U10.20 (AGND), U10.25 (PGND), U10.26 (PGND), U10.31 (PGND), U10.32 (PGND), U10.33 (EP), U10.5 (DGND), U9.20 (AGND), U9.25 (PGND), U9.26 (PGND), U9.31 (PGND), U9.32 (PGND), U9.33 (EP), U9.5 (DGND); no longer C51.2, C52.2, C65.2, C66.2
- net at C52.1: now also JP5.2, L5.2, U9.30 (OUT_A-)
- net at C61.1: now also J5.4 (Pin_4), JP8.2, L7.1
- net AMP_FAULT1: now reaches R43.2
- net AMP_FAULT1: now also U10.9 (GPIO0)
- net at C71.1: now also JP1.2, L9.2, U10.30 (OUT_A-)
- net at C50.1: now also JP5.1, L4.1, U9.2 (OUT_A+); no longer R45.2
- net at C53.1: now also J5.2 (Pin_2), JP6.2, L5.1; no longer R44.2
- net at R45.1: now also R41.1, U10.14 (SDIN)
- net at R46.1: now also U10.8 (ADR); no longer C47.1
- net at R41.2: now also U9.11 (GPIO2)
- net +3.0VA: no longer names the net of R40.1
- net +3.0VA: now also U9.8 (ADR); no longer C65.1
- removed net GNDA: C46.2, C50.2, C53.2, C70.2, C71.2, R42.2
- removed net MIC-DET: R40.2, R41.1
- new net: C56.1, JP7.1, L6.1, U9.23 (OUT_B+)
- new net: C60.1, JP7.2, L7.2, U9.27 (OUT_B-)
- new net: C51.2, J5.1 (Pin_1), JP6.1, L4.2
- new net: C57.2, J5.3 (Pin_3), JP8.1, L6.2
- new net: C50.2, U9.1 (BST_A+)
- new net: C45.2, U9.18 (GVDD)
- new net: C46.2, U9.19 (AVDD)
- new net: C56.2, U9.24 (BST_B+)
- new net: C60.2, U9.28 (BST_B-)
- new net: C52.2, U9.29 (BST_A-)
- new net: C43.2, C44.2, U9.6 (DVDD)
- new net: C47.2, U9.7 (VR_DIG)
- new net: C69.2, U10.1 (BST_A+)
- new net: C64.2, U10.18 (GVDD)
- new net: C65.2, U10.19 (AVDD)
- new net: C69.1, JP1.1, L8.1, U10.2 (OUT_A+)
- new net: C75.1, JP3.1, L10.1, U10.23 (OUT_B+)
- new net: C75.2, U10.24 (BST_B+)
- new net: C79.1, JP3.2, L11.2, U10.27 (OUT_B-)
- new net: C79.2, U10.28 (BST_B-)
- new net: C71.2, U10.29 (BST_A-)
- new net: C62.2, C63.2, U10.6 (DVDD)
- new net: C66.2, U10.7 (VR_DIG)
- new net: C70.2, J6.1 (Pin_1), JP2.1, L8.2
- new net: C72.1, J6.2 (Pin_2), JP2.2, L9.1
- new net: C76.2, J6.3 (Pin_3), JP4.1, L10.2
- new net: C80.1, J6.4 (Pin_4), JP4.2, L11.1
- new net AMP_FAULT0: R38.2, U9.9 (GPIO0)
- new net AMP_MUTE0: R37.2, U9.10 (GPIO1)
- new net AMP_MUTE1: R42.2, U10.10 (GPIO1)
- new net AMP_PDN0: R39.2, U9.17 (~PDN)
- new net AMP_PDN1: R44.2, U10.17 (~PDN)
- new net I2C1_SCL: U10.16 (SCL), U9.16 (SCL)
- new net I2C1_SDA: U10.15 (SDA), U9.15 (SDA)
- new net PCM_BCLK: U10.13 (SCLK), U9.13 (SCLK)
- new net PCM_DOUT: R45.2, U9.14 (SDIN)
- new net PCM_LRCLK: U10.12 (LRCLK), U9.12 (LRCLK)
- new net VBUS: C48.1, C49.1, C54.1, C55.1, C58.1, C59.1, C67.1, C68.1, C73.1, C74.1, C77.1, C78.1, U10.21 (PVDD), U10.22 (PVDD), U10.3 (PVDD), U10.4 (PVDD), U9.21 (PVDD), U9.22 (PVDD), U9.3 (PVDD), U9.4 (PVDD)
- no-connect marks 6 -> 0
Other:
- note added: "ADR: 0x48C"
- note added: "ADR: 0x4D"
- note removed: "0x1B"

Commit message: V1.0 order release
Connections:
- net +3V3: now also C43.2, C44.2, C62.2, C63.2, U10.6 (DVDD), U9.6 (DVDD)
Changed lines of the file:
@@
 	0    1    1    0
 $EndComp
+$Comp
+L power:+3V3 #PWR?
+U 1 1 604259A9
+P 5650 3850
+F 0 "#PWR?" H 5650 3700 50  0001 C CNN
+F 1 "+3V3" H 5665 4023 50  0000 C CNN
+F 2 "" H 5650 3850 50  0001 C CNN
+F 3 "" H 5650 3850 50  0001 C CNN
+	1    5650 3850
+	1    0    0    -1
+$EndComp
+Connection ~ 5650 3850
+$Comp
+L power:+3V3 #PWR?
+U 1 1 60426587
+P 5650 950
+F 0 "#PWR?" H 5650 800 50  0001 C CNN
+F 1 "+3V3" H 5665 1123 50  0000 C CNN
+F 2 "" H 5650 950 50  0001 C CNN
+F 3 "" H 5650 950 50  0001 C CNN
+	1    5650 950
+	1    0    0    -1
+$EndComp
+Connection ~ 5650 950
 $EndSCHEMATC
