File: OtterCastAmp.kicad_pcb (KiCad board)
At the start: 4 copper layers, 50 x 49.3 mm, 226 parts, among them J1 UART, J2 SD, J3 USB, J4 OTG, J5 PJ-3270, J6 PJ-3270, J7 PJ-3270, J8 49F-1201GYD2NL, Q1 DTA114YKA, SW3 RST, U1 AllWinner-S3(FBGA-234), U3 AXP209(QFN-48), U4 SY8089AAAC, U5 SY6280AAC, U6 SSM2603, U7 AP6236, X1 26Mhz TCXO, Y1 12.288Mhz, Y2 32.768kHz, Y3 24MHz

Commit message: started layout
Parts:
- removed FB2, FB3: FERRET, otter:R_0805
- removed G***: LOGO, otter:OtterCastAudioV2_hw_v2.1
- removed G***: LOGO, otter:OtterCastAudioV2_silk_1
- removed G***: LOGO, otter:OtterCastAudioV2_silk_3
- removed G***: LOGO, otter:OtterCastAudioV2_silk_amp_out
- removed G***: LOGO, otter:OtterCastAudioV2_silk_line_out
- removed G***: LOGO, otter:OtterCastAudioV2_silk_line_in
- removed G***: LOGO, otter:OtterCastAudioV2_silk_by
- removed G***: LOGO, otter:OtterCastAudioV2_silk_status
- removed G***: LOGO, otter:OtterCastAudioV2_silk_power
- removed G***: LOGO, otter:OtterCastAudioV2_silk_2
- removed J7: PJ-3270, otter:PJ-3270
- removed J8: 49F-1201GYD2NL, otter:49F-1201GYDXNL
- removed MK1: Mic, otter:B4013AM422-42
- removed R60: 47k, otter:R_0402
- removed R61: 100, otter:R_0402
- removed R82, R83: 240, otter:R_0402
- removed R84: 10M, otter:R_0402
- removed R86: 5k1, otter:R_0402
- removed R87, R88: 2k2, otter:R_0402
- removed R89: 6k04, otter:R_0402
- removed R90, R91, R92, R93: 51, otter:R_0402
- removed SW3: RST, otter:SW_SPST_PTS810
- removed X1: 26Mhz TCXO, otter:2016_SMD_CRYSTAL
- added C105: 18p, otter:C_0402, F.Cu at (183.9, 84.1)
- added C106: 18p, otter:C_0402, F.Cu at (183.9, 86.7)
- added C107: 10u, otter:C_0603, F.Cu at (174.8, 85.9)
- added C108: 100n, otter:C_0402, F.Cu at (184.4, 93.2)
- added C109: 18p, otter:C_0402, F.Cu at (180.3, 85.1)
- added C111: 100n, otter:C_0402, F.Cu at (191.2, 89.0)
- added C113: 18p, otter:C_0402, F.Cu at (175.5, 84.5)
- added C114: 100n 50V, otter:C_0603, F.Cu at (198.7, 81.4)
- added C115: 22u 50V, Capacitor_SMD:C_1206_3216Metric, F.Cu at (184.4, 80.8)
- added C116: 470u 35V, Capacitor_SMD:CP_Elec_10x10.5, F.Cu at (188.3, 70.0)
- added C117: 18p, otter:C_0402, F.Cu at (167.1, 108.2)
- added C118: 18p, otter:C_0402, F.Cu at (167.1, 109.8)
- added C119: 100n, otter:C_0402, F.Cu at (173.5, 121.8)
- added C120: 100n, otter:C_0402, F.Cu at (173.5, 123.3)
- added C121: 100n, otter:C_0402, F.Cu at (175.9, 121.8)
- added C122: 100n, otter:C_0402, F.Cu at (175.9, 123.3)
- added C123: 10u, otter:C_0603, F.Cu at (170.7, 76.6)
- added C124: 10u, otter:C_0603, F.Cu at (169.4, 76.6)
- added C125: 10u, otter:C_0603, F.Cu at (168.1, 76.6)
- added C126: 10u, otter:C_0603, F.Cu at (166.8, 76.6)
- added C127: 10u, otter:C_0603, F.Cu at (170.7, 79.1)
- added C40: 1u, otter:C_0402, F.Cu at (175.4, 65.7)
- added C79: 470n 25V, otter:C_0603, F.Cu at (125.2, 109.9)
- added C80: 680n 50V, Capacitor_SMD:C_1206_3216Metric, F.Cu at (110.2, 115.1)
- added C81: 10u, otter:C_0603, F.Cu at (206.4, 105.2)
- added C84: 100n, otter:C_0402, F.Cu at (213.8, 100.4)
- added C86: 1p, otter:C_0402, F.Cu at (231.6, 145.1)
- added C87: 1p, otter:C_0402, F.Cu at (214.0, 105.2)
- added C91: 100n, otter:C_0402, F.Cu at (158.2, 71.8)
- added C99: 10u, otter:C_0603, F.Cu at (183.7, 116.3)
- added D7: LED, otter:LED_0603_1608Metric, F.Cu at (158.7, 77.5)
- added H1: 3.2mm, MountingHole:MountingHole_3.2mm_M3_Pad_Via, F.Cu at (130.0, 80.0)
- added H2: 3.2mm, MountingHole:MountingHole_3.2mm_M3_Pad_Via, F.Cu at (130.0, 120.0)
- added IC1: EMMC04G-S100-B08U, lib:MICRON_EMMC_153, F.Cu at (176.7, 103.8)
- added J10: FH26W-33S-0.3SHW, Connector_FFC-FPC:Molex_502250-3391_2Rows-33Pins-1MP_P0.60mm_Horizontal, F.Cu at (153.9, 129.2)
- added J9: PJ-3270, otter:PJ-3270, F.Cu at (189.7, 50.6)
- added JP1: PBTL, Jumper:SolderJumper-2_P1.3mm_Open_Pad1.0x1.5mm, F.Cu at (124.7, 120.3)
- added JP2: PBTL, Jumper:SolderJumper-2_P1.3mm_Open_Pad1.0x1.5mm, F.Cu at (117.5, 62.1)
- added JP3: PBTL, Jumper:SolderJumper-2_P1.3mm_Open_Pad1.0x1.5mm, F.Cu at (124.0, 107.8)
- added JP4: PBTL, Jumper:SolderJumper-2_P1.3mm_Open_Pad1.0x1.5mm, F.Cu at (107.5, 62.1)
- added JP5: PBTL, Jumper:SolderJumper-2_P1.3mm_Open_Pad1.0x1.5mm, F.Cu at (124.0, 92.2)
- added JP6: PBTL, Jumper:SolderJumper-2_P1.3mm_Open_Pad1.0x1.5mm, F.Cu at (140.0, 62.1)
- added JP7: PBTL, Jumper:SolderJumper-2_P1.3mm_Open_Pad1.0x1.5mm, F.Cu at (124.7, 79.7)
- added JP8: PBTL, Jumper:SolderJumper-2_P1.3mm_Open_Pad1.0x1.5mm, F.Cu at (130.0, 62.1)
- added L10: 10u, otter:L_10.4x10.4_H4.8, F.Cu at (117.3, 105.5)
- added L11: 10u, otter:L_10.4x10.4_H4.8, F.Cu at (117.3, 116.5)
- added L12: 2.2nH, otter:L_0402, F.Cu at (231.6, 143.5)
- added L13: 2.2uH, otter:Inductor_4040, F.Cu at (167.9, 85.8)
- added L6: 10u, otter:L_10.4x10.4_H4.8, F.Cu at (130.0, 71.0)
- added L7: 10u, otter:L_10.4x10.4_H4.8, F.Cu at (117.3, 72.5)
- added L8: 10u, otter:L_10.4x10.4_H4.8, F.Cu at (130.0, 129.0)
- added L9: 10u, otter:L_10.4x10.4_H4.8, F.Cu at (117.3, 127.5)
- added R19: 68k, otter:R_0402, F.Cu at (162.7, 82.4)
- added R20: 47k, otter:R_0402, F.Cu at (192.5, 76.0)
- added R5: 2.2k, otter:R_0402, F.Cu at (189.4, 141.6)
- added R53: 22, otter:R_0402, F.Cu at (167.2, 92.9)
- added R55: DNP, otter:R_0402, F.Cu at (161.3, 85.5)
- added R56: DNP, otter:R_0402, F.Cu at (162.2, 85.5)
- added R57: 47k, otter:R_0402, F.Cu at (223.7, 102.9)
- added SW1: CONFIG, Button_Switch_THT:SW_Tactile_SPST_Angled_PTS645Vx58-2LFS, F.Cu at (91.0, 73.0)
- added U10: TAS5825MRHB, Package_DFN_QFN:Texas_S-PVQFN-N32_EP3.45x3.45mm, F.Cu at (130.0, 110.0)
- added U11: AP6236, otter:LGA_44_12x12mm_0.9mm, F.Cu at (159.5, 92.9)
- added U2: LM75B, Package_SO:VSSOP-8_3.0x3.0mm_P0.65mm, F.Cu at (130.0, 100.0)
- added U9: TAS5825MRHB, Package_DFN_QFN:Texas_S-PVQFN-N32_EP3.45x3.45mm, F.Cu at (130.0, 90.0)
- AE1: value KH-5220-A56_U.FL -> u.FL; footprint otter:KH-5220-A56 -> Connector_Coaxial:U.FL_Molex_MCRF_73412-0110_Vertical; moved to F.Cu
- C10: value 47u -> 10u; footprint otter:C_0805 -> otter:C_0603
- C101, C15, C21, C35, C36, C37, C44, C8, C83, C88: value 100n -> 10u; footprint otter:C_0402 -> otter:C_0603
- C104: value 1n -> 100n; footprint otter:C_0805 -> otter:C_0402
- C11, C42, C43, C5: value 47u -> 100n; footprint otter:C_0805 -> otter:C_0402
- C12: value 1n -> 10u; footprint otter:C_0402 -> otter:C_0603
- C13: value 1n -> 10u; footprint otter:C_0805 -> otter:C_0603
- C16, C17, C19, C24, C29, C30, C39, C90: value 10u -> 100n; footprint otter:C_0603 -> otter:C_0402
- C18: value 100n -> 3.3n
- C2: value 470n -> DNP
- C32: moved to F.Cu
- C38: value 100n -> 1u 25V; footprint otter:C_0402 -> otter:C_0603; moved to F.Cu
- C41: value 10u -> 1u; footprint otter:C_0603 -> otter:C_0402
- C45: value 47u -> 1u; footprint otter:C_0805 -> otter:C_0402
- C46: value 220p -> 1u
- C47: value 1n -> 1u
- C48: value 10u -> 100n 50V
- C49: value DNP -> 100n 50V; footprint otter:C_0402 -> otter:C_0603; moved to F.Cu
- C50, C71: value 220p -> 470n 25V; footprint otter:C_0402 -> otter:C_0603
- C51: value 18p -> 680n 50V; footprint otter:C_0402 -> Capacitor_SMD:C_1206_3216Metric
- C52: value 18p -> 470n 25V; footprint otter:C_0402 -> otter:C_0603
- C53, C70: value 220p -> 680n 50V; footprint otter:C_0402 -> Capacitor_SMD:C_1206_3216Metric
- C54, C55: value 10u -> 22u 50V; footprint otter:CP_EIA-3216-10 -> Capacitor_SMD:C_1206_3216Metric
- C56, C60, C69: value 10u -> 470n 25V; footprint otter:CP_EIA-3216-10 -> otter:C_0603
- C57: value 10u -> 680n 50V; footprint otter:CP_EIA-3216-10 -> Capacitor_SMD:C_1206_3216Metric
- C58, C59: value 100n -> 470u 35V; footprint otter:C_0402 -> Capacitor_SMD:CP_Elec_10x10.5
- C61, C76: value 100n -> 680n 50V; footprint otter:C_0402 -> Capacitor_SMD:C_1206_3216Metric
- C62: value 10u -> 100n; footprint otter:CP_EIA-3216-10 -> otter:C_0402
- C63: footprint otter:CP_EIA-3216-10 -> otter:C_0603
- C64: value 10u -> 1u; footprint otter:CP_EIA-3216-10 -> otter:C_0402
- C65, C66: value 100n -> 1u
- C67, C68: value 100u -> 100n 50V; footprint otter:CP_EIA-3528-12 -> otter:C_0603
- C7: value 100n -> 10n
- C72: value 10u -> 680n 50V; footprint otter:C_0603 -> Capacitor_SMD:C_1206_3216Metric
- C73: value 100n -> 22u 50V; footprint otter:C_0402 -> Capacitor_SMD:C_1206_3216Metric
- C74: value 10u -> 22u 50V; footprint otter:C_0603 -> Capacitor_SMD:C_1206_3216Metric
- C75: value 1p -> 470n 25V; footprint otter:C_0402 -> otter:C_0603
- C77: value 1p -> 470u 35V; footprint otter:C_0402 -> Capacitor_SMD:CP_Elec_10x10.5
- C78: value 10p -> 470u 35V; footprint otter:C_0402 -> Capacitor_SMD:CP_Elec_10x10.5
- C85: value 100n -> 10p
- C9: value 2.2u -> 10u
- C92: value 10u -> 1u 25V; moved to F.Cu
- C93, C94: value 18p -> 100n
- C95: value 10u -> 1u 25V
- C96: value 18p -> 1n 2kV; footprint otter:C_0402 -> Capacitor_SMD:C_1206_3216Metric
- C97: value 18p -> 10u; footprint otter:C_0402 -> otter:C_0603
- D3: value LED -> SMAJ22A; footprint LED_SMD:LED_0603_1608Metric_Castellated -> Diode_SMD:D_SMA
- D4: value P6SMB6.8CA -> SMAJ22A; footprint Diode_SMD:D_SMB -> Diode_SMD:D_SMA
- J1: value UART -> HR911105A; footprint otter:PinHeader_1x04_P2.00mm_Vertical_nosilk_center -> Connector_RJ:RJ45_Hanrun_HR911105A
- J2: value SD -> Micro_SD_Card; footprint Connector_Card:microSD_HC_Hirose_DM3D-SF -> ST-TF-003A:SUNTECH_ST-TF-003A
- J4: value OTG -> UART1; footprint otter:PinHeader_1x04_P2.00mm_Vertical_nosilk_center -> Connector_PinHeader_2.54mm:PinHeader_1x03_P2.54mm_Vertical
- J5, J6: value PJ-3270 -> C475204; footprint otter:PJ-3270 -> otter:C475204
- L1: value 2.2uH -> 15uH; footprint Inductor_SMD:L_Taiyo-Yuden_MD-3030 -> otter:L_10.4x10.4_H4.8
- L2, L3: value 2.2uH -> 2u2; footprint Inductor_SMD:L_Taiyo-Yuden_MD-3030 -> otter:Inductor_4040
- L4: value 2.2uH -> 10u; footprint Inductor_SMD:L_Taiyo-Yuden_MD-3030 -> otter:L_10.4x10.4_H4.8
- L5: value 2.2uH -> 10u; footprint otter:L_0402 -> otter:L_10.4x10.4_H4.8
- Q1: value DTA114YKA -> IRF8736; footprint Package_TO_SOT_SMD:SOT-23 -> Package_SO:SOIC-8_3.9x4.9mm_P1.27mm
- R1: value 100 -> 47k
- R12, R59, R64: value 47k -> 22
- R14, R4: value 5k1 -> 47k
- R15, R2: value 22 -> 47k
- R16, R78: value 200k -> 100k
- R17: value 2.2k -> 100k
- R18: value 47k -> 31.25k
- R21: value 200k -> 10k
- R22: value DNP -> 5.6k
- R23: value DNP -> 100k
- R24: value 5k1 -> 68k
- R25, R3: value 5k1 -> 22
- R26: value 47k -> 100k
- R27: value 0R -> 100R; footprint otter:R_0805 -> otter:R_0402
- R29: value DNP -> 22k
- R30: value 5.1k -> 1k
- R31: value 3.3k -> DNP
- R32: value 100 -> DNP
- R33: value 100 -> 100k
- R34: value 22 -> 100k
- R35: value 5k1 -> 100k
- R36: value 5k1 -> 2.2k
- R37: value 2k2 -> 10k
- R38: value 3k9 -> 10k
- R39: value 5k1 -> 10k
- R40: value 200k -> 0R
- R41: value 2k2 -> 0R
- R42, R65: value 47k -> 10k
- R43: value 680 -> 10k
- R44: value 0 -> 10k
- R45: value 0 -> DNP
- R46: value 0 -> 1k
- R47, R52: value DNP -> 47k
- R48, R49, R50, R51: value 2.2k -> 47k
- R54: value 22 -> DNP
- R6: value DNP -> 2.2k
- R62: value 100 -> 2.2k
- R63, R7, R8: value 47k -> 2.2k
- R66, R67, R69: value DNP -> 51
- R70: value 47k -> 51
- R71: value 47k -> DNP
- R72, R73: value 47k -> 200k
- R74: value 47k -> 6k04
- R75: value 47k -> 5k1
- R76: value 22 -> 10M
- R77: value 22 -> 2k2
- R80: value 2k2 -> 240
- R81: value 22 -> 240
- U3: value AXP209(QFN-48) -> SY8089AAAC; footprint otter:QFN-48-1EP_6x6mm_P0.4mm_EP4.05x4.05mm -> Package_TO_SOT_SMD:SOT-23-5
- U4: value SY8089AAAC -> MP2303; footprint Package_TO_SOT_SMD:SOT-23-5 -> Package_SO:SOIC-8-1EP_3.9x4.9mm_P1.27mm_EP2.29x3mm
- U5: value SY6280AAC -> SY8089AAAC
- U6: value SSM2603 -> MIC5501-3.0YM5; footprint otter:LFCSP-28-5x5mm-0.5mm-EP3.14x3.14mm -> Package_TO_SOT_SMD:SOT-23-5
- U7: value AP6236 -> STUSB4500; footprint otter:LGA_44_12x12mm_0.9mm -> Package_DFN_QFN:QFN-24-1EP_4x4mm_P0.5mm_EP2.7x2.7mm
- Y1: value 12.288Mhz -> 32.768kHz; footprint otter:Oscillator_3225 -> otter:Crystal_SMD_3215-2Pin_3.2x1.5mm
- Y2: value 32.768kHz -> 24MHz; footprint otter:Crystal_SMD_3215-2Pin_3.2x1.5mm -> otter:Oscillator_3225
- Y3: value 24MHz -> 26MHz
- moved R4 143.8 mm to (229.1, 105.3), turned to 0 degrees
- moved C34 140.5 mm to (234.0, 117.9), turned to 0 degrees
- moved C31 132.4 mm to (227.4, 118.6), turned to 0 degrees
- moved C35 128.9 mm to (224.4, 123.2), turned to 0 degrees
- moved C33 128.3 mm to (223.6, 127.0), turned to 0 degrees
- moved C24 126.4 mm to (234.2, 116.1), turned to 0 degrees
- moved C13 126.3 mm to (216.8, 128.2), turned to 0 degrees
- moved C30 124.7 mm to (214.0, 130.4), turned to 0 degrees
- moved C29 122.4 mm to (230.9, 119.9), turned to 0 degrees
- moved C82 119.4 mm to (213.9, 102.0), turned to 0 degrees
- moved C32 119.3 mm to (211.6, 130.4), turned to 0 degrees
- moved C11 118.8 mm to (231.3, 116.1)
- moved C12 115.9 mm to (232.7, 113.9)
- moved R68 115.9 mm to (190.7, 119.8)
- moved C5 115.8 mm to (231.5, 102.1), turned to 0 degrees
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Connections:
- net PB6\TWI0-SCK renamed I2C0_SCL
- net PB7\TWI0-SDA renamed I2C0_SDA
- net PB8\TWI1-SCK renamed UART0_TX
- net PB9\TWI1-SDA renamed UART0_RX
- C10 pad 1: IPS -> +1V5
- C100 pad 1: GND -> +3.0VA
- C100 pad 2: Net-(C100-Pad2) -> GND
- C101 pad 1: GND -> +3V3
- C101 pad 2: Net-(C101-Pad2) -> GND
- C102 pad 1: GND -> Net-(C102-Pad1)
- C102 pad 2: Net-(C102-Pad2) -> GND
- C103 pad 1: GND -> +3V3
- C103 pad 2: Net-(C103-Pad2) -> GND
- C104 pad 2: GND -> +1V5
- C11 pad 1: +5V -> +1V5
- C12 pad 1: Net-(C12-Pad1) -> +1V5
- C13 pad 1: Net-(C13-Pad1) -> +1V5
- C14 pad 1: +5V -> +1V5
- C15 pad 1: Net-(C15-Pad1) -> +1V5
- C16 pad 1: IPS -> +3V3
- C17 pad 1: IPS -> Net-(C17-Pad1)
- C18 pad 1: +1.1V -> Net-(C18-Pad1)
- C18 pad 2: GND -> Net-(C18-Pad2)
- C19 pad 1: IPS -> +1.1V
- C2 pad 1: RESETn -> SDC2_CLK
- C20 pad 1: IPS -> +1.1V
- C23 pad 1: +3V3 -> +1.1V
- C24 pad 1: IPS -> +1.1V
- C25 pad 1: +3.3V_RTC -> +1.1V
- C26 pad 1: +3.0VA -> +1.1V
- C27 pad 1: +1V2 -> +1.1V
- C28 pad 1: IPS -> +1.1V
- C29 pad 1: +2V8 -> +1.1V
- C30 pad 1: IPS -> +1.1V
- C31 pad 1: VCC-DDR -> +1.1V
- C32 pad 1: VCC-DDR -> +1V5
- C33 pad 1: +1.1V -> +1V5
- C34 pad 1: VCC-DDR -> +1V5
- C35 pad 1: +1.1V -> +1V5
- C36 pad 1: +1.1V -> +3V3
- C37 pad 1: VCC-DDR -> +3.0VA
- C38 pad 1: +3V3 -> GND
- C38 pad 2: GND -> Net-(C38-Pad2)
- C39 pad 1: +1.1V -> VBUS
- C39 pad 2: GND -> Net-(C39-Pad2)
- C4 pad 1: Net-(C4-Pad1) -> Net-(C3-Pad1)
- C41 pad 1: VCC-DDR -> GND
- C41 pad 2: GND -> Net-(C41-Pad2)
- C42 pad 1: +5V -> +3V3
- C43 pad 1: +5V_USBOTG -> GND
- C43 pad 2: GND -> Net-(C43-Pad2)
- C44 pad 1: USB-VBUSDET -> GND
- C44 pad 2: GND -> Net-(C43-Pad2)
- C45 pad 1: +5V_USBOTG -> GND
- C45 pad 2: GND -> Net-(C45-Pad2)
- C46 pad 1: Net-(C46-Pad1) -> GND
- C46 pad 2: GNDA -> Net-(C46-Pad2)
- C47 pad 1: Net-(C47-Pad1) -> GND
- C47 pad 2: Net-(C46-Pad1) -> Net-(C47-Pad2)
- C48 pad 1: Net-(C48-Pad1) -> VBUS
- C49 pad 1: Net-(C48-Pad1) -> VBUS
- C5 pad 1: IPS -> GPIO_BTN
- C50 pad 2: GNDA -> Net-(C50-Pad2)
- C51 pad 1: Net-(C51-Pad1) -> GND
- C51 pad 2: GND -> Net-(C51-Pad2)
- C52 pad 2: GND -> Net-(C52-Pad2)
- C53 pad 2: GNDA -> GND
- C54 pad 1: Net-(C54-Pad1) -> VBUS
- C54 pad 2: GNDA -> GND
- C55 pad 1: Net-(C55-Pad1) -> VBUS
- C55 pad 2: GNDA -> GND
- C56 pad 2: Net-(C53-Pad1) -> Net-(C56-Pad2)
- C57 pad 1: Net-(C57-Pad1) -> GND
- C57 pad 2: Net-(C50-Pad1) -> Net-(C57-Pad2)
- C58 pad 1: Net-(C54-Pad1) -> VBUS
- C58 pad 2: GNDA -> GND
- C59 pad 1: Net-(C55-Pad1) -> VBUS
- C59 pad 2: GNDA -> GND
- C6 pad 1: +5V_USBOTG -> Net-(C6-Pad1)
- C60 pad 1: +3.0VA -> Net-(C60-Pad1)
- C60 pad 2: GND -> Net-(C60-Pad2)
- C62 pad 1: +3V3 -> GND
- C62 pad 2: GND -> Net-(C62-Pad2)
- C63 pad 1: Net-(C63-Pad1) -> GND
- C63 pad 2: Net-(C63-Pad2) -> Net-(C62-Pad2)
- C64 pad 1: Net-(C64-Pad1) -> GND
- C65 pad 1: +3.0VA -> GND
- C65 pad 2: GND -> Net-(C65-Pad2)
- C66 pad 1: +3V3 -> GND
- C66 pad 2: GND -> Net-(C66-Pad2)
- C67 pad 1: Net-(C67-Pad1) -> VBUS
- C67 pad 2: Net-(C67-Pad2) -> GND
- C68 pad 1: Net-(C68-Pad1) -> VBUS
- C68 pad 2: Net-(C68-Pad2) -> GND
- C69 pad 1: Net-(C61-Pad1) -> Net-(C69-Pad1)
- C69 pad 2: GND -> Net-(C69-Pad2)
- C7 pad 1: +2.5V -> Net-(C7-Pad1)
- C7 pad 2: GND -> Net-(C7-Pad2)
- C70 pad 1: Net-(C68-Pad2) -> GND
- C70 pad 2: GNDA -> Net-(C70-Pad2)
- C71 pad 1: Net-(C67-Pad2) -> Net-(C71-Pad1)
- C71 pad 2: GNDA -> Net-(C71-Pad2)
- C72 pad 1: +3V3 -> Net-(C72-Pad1)
- C73 pad 1: +3V3 -> VBUS
- C74 pad 1: +3V3 -> VBUS
- C75 pad 1: GND -> Net-(C75-Pad1)
- C75 pad 2: Net-(AE1-Pad1) -> Net-(C75-Pad2)
- C76 pad 1: +3V3 -> GND
- C76 pad 2: GND -> Net-(C76-Pad2)
- C77 pad 1: GND -> VBUS
- C77 pad 2: Net-(C77-Pad2) -> GND
- C78 pad 1: Net-(C77-Pad2) -> VBUS
- C78 pad 2: Net-(C78-Pad2) -> GND
- C8 pad 1: IPS -> +3V3
- C82 pad 1: Net-(C82-Pad1) -> +3V3
- C82 pad 2: VCC-DDR -> GND
- C83 pad 1: Net-(C82-Pad1) -> +3V3
- C85 pad 2: GND -> Net-(C85-Pad2)
- C88 pad 1: Net-(C82-Pad1) -> Net-(C88-Pad1)
- C89 pad 1: +3.0VA -> Net-(C88-Pad1)
- C9 pad 1: GND -> +1V5
- C9 pad 2: Net-(C9-Pad2) -> GND
- C90 pad 1: Net-(C90-Pad1) -> GND
- C90 pad 2: GND -> Net-(C90-Pad2)
- C92 pad 1: +1.1V -> LINE_L
- C92 pad 2: GND -> Net-(C92-Pad2)
- C93 pad 1: Net-(C93-Pad1) -> GND
- C93 pad 2: GND -> Net-(C93-Pad2)
- C94 pad 1: Net-(C94-Pad1) -> GND
- C94 pad 2: GND -> Net-(C94-Pad2)
- C95 pad 1: +3V3 -> Net-(C95-Pad1)
- C95 pad 2: GND -> LINE_R
- C97 pad 1: Net-(C97-Pad1) -> +3V3
- C98 pad 1: +3.3V_RTC -> Net-(C98-Pad1)
- D3 pad 1: GND -> Net-(C38-Pad2)
- D3 pad 2: Net-(D3-Pad2) -> GND
- D4 pad 1: +5V -> VBUS
- D6 pad 1: USB-D_P -> USB-D_N
- D6 pad 2: USB-D_N -> USB-D_P
- FB1 pad 2: Net-(C4-Pad1) -> Net-(C6-Pad1)
- J1 pad 1: GND -> EPHY_TX_P
- J1 pad 2: Net-(D5-Pad2) -> EPHY_TX_N
- J1 pad 3: Net-(D5-Pad1) -> EPHY_RX_P
- J1 pad 4: +3V3 -> Net-(C91-Pad2)
- J2 pad 1: SDC0-D2 -> SDC0_D2
- J2 pad 2: SDC0-D3 -> SDC0_D3
- J2 pad 3: SDC0-CMD -> SDC0_CMD
- J2 pad 4: Net-(C4-Pad1) -> Net-(C6-Pad1)
- J2 pad 5: SDC0-CLK -> SDC0_CLK
- J2 pad 7: SDC0-D0 -> SDC0_D0
- J2 pad 8: SDC0-D1 -> SDC0_D1
- J3 pad A4: +5V -> Net-(C38-Pad2)
- J3 pad A5: Net-(J3-PadA5) -> Net-(D5-Pad2)
- J3 pad A9: +5V -> Net-(C38-Pad2)
- J3 pad B4: +5V -> Net-(C38-Pad2)
- J3 pad B5: Net-(J3-PadB5) -> Net-(D5-Pad1)
- J3 pad B9: +5V -> Net-(C38-Pad2)
- J3 pad S1: Net-(C13-Pad1) -> GND
- J4 pad 2: USB-D_P -> UART1_TX
- J4 pad 3: USB-D_N -> UART1_RX
- J5 pad 2: Net-(J5-Pad2) -> Net-(C53-Pad1)
- J5 pad 3: Net-(J5-Pad3) -> Net-(C57-Pad2)
- J5 pad 4: GNDA -> Net-(C61-Pad1)
- J6 pad 2: Net-(C68-Pad2) -> Net-(C72-Pad1)
- J6 pad 3: Net-(J6-Pad3) -> Net-(C76-Pad2)
- J6 pad 4: GNDA -> Net-(C80-Pad1)
- L1 pad 1: Net-(L1-Pad1) -> Net-(C7-Pad1)
- L2 pad 2: +1.1V -> +1V5
- L3 pad 2: VCC-DDR -> +1.1V
- L4 pad 1: Net-(C48-Pad1) -> Net-(C50-Pad1)
- L4 pad 2: Net-(L4-Pad2) -> Net-(C51-Pad2)
- L5 pad 1: Net-(AE1-Pad1) -> Net-(C53-Pad1)
- L5 pad 2: Net-(C77-Pad2) -> Net-(C52-Pad1)
- Q1 pad 1: Net-(Q1-Pad1) -> Net-(C38-Pad2)
- Q1 pad 2: IPS -> Net-(C38-Pad2)
- Q1 pad 3: Net-(Q1-Pad3) -> Net-(C38-Pad2)
- R1 pad 1: Net-(D5-Pad2) -> +3V3
- R1 pad 2: UART1_RX -> SDC2_CMD
- R10 pad 1: SDC0-CLK -> SDC0_D3
- R11 pad 1: SDC0-D0 -> SDC0_CMD
- R12 pad 1: SDC0-D1 -> Net-(R12-Pad1)
- R12 pad 2: +3V3 -> BT-DIS-N
- R13 pad 1: SDC0-DET# -> SDC0_CLK
- R14 pad 1: Net-(D3-Pad2) -> SDC0_D0
- R14 pad 2: +5V -> +3V3
- R15 pad 1: Net-(R15-Pad1) -> SDC0_D1
- R15 pad 2: GND -> +3V3
- R16 pad 1: Net-(R16-Pad1) -> +1V5
- R16 pad 2: GND -> Net-(R16-Pad2)
- R17 pad 1: Net-(Q1-Pad3) -> Net-(R17-Pad1)
- R17 pad 2: GND -> VBUS
- R18 pad 1: /Power/NMI -> +3V3
- R18 pad 2: +3.3V_RTC -> Net-(R18-Pad2)
- R2 pad 1: Net-(R2-Pad1) -> +3V3
- R2 pad 2: BT-DIS-N -> SDC2_RST
- R21 pad 1: Net-(C13-Pad1) -> Net-(R18-Pad2)
- R22 pad 1: Net-(J3-PadA7) -> Net-(C18-Pad1)
- R22 pad 2: USB-D_N -> GND
- R23 pad 1: Net-(J3-PadA6) -> +1.1V
- R23 pad 2: USB-D_P -> Net-(R23-Pad2)
- R24 pad 1: Net-(J3-PadA5) -> Net-(R23-Pad2)
- R25 pad 1: Net-(J3-PadB5) -> Net-(R25-Pad1)
- R26 pad 1: +3.3V_RTC -> Net-(Q1-Pad4)
- R26 pad 2: RESETn -> Net-(C38-Pad2)
- R27 pad 1: GND -> Net-(C39-Pad2)
- R27 pad 2: GNDA -> Net-(Q1-Pad4)
- R28 pad 1: VINT -> Net-(R28-Pad1)
- R28 pad 2: Net-(R28-Pad2) -> Net-(C38-Pad2)
- R29 pad 1: GND -> Net-(R29-Pad1)
- R29 pad 2: Net-(R28-Pad2) -> Net-(Q1-Pad4)
- R3 pad 1: GPIO_LED1 -> SDC2_CLK
- R3 pad 2: Net-(D1-Pad2) -> Net-(R3-Pad2)
- R30 pad 1: VCC-DDR -> Net-(R30-Pad1)
- R30 pad 2: Net-(R30-Pad2) -> VBUS
- R31 pad 1: Net-(R30-Pad2) -> Net-(J3-PadA7)
- R31 pad 2: Net-(R31-Pad2) -> USB-D_N
- R32 pad 1: Net-(R31-Pad2) -> Net-(J3-PadA6)
- R32 pad 2: GND -> USB-D_P
- R33 pad 1: Net-(D5-Pad1) -> GND
- R33 pad 2: UART1_TX -> Net-(R33-Pad2)
- R34 pad 1: Net-(R34-Pad1) -> GND
- R34 pad 2: GND -> Net-(R34-Pad2)
- R35 pad 1: USB-DRV -> Net-(R35-Pad1)
- R36 pad 1: Net-(R36-Pad1) -> +3V3
- R36 pad 2: GND -> I2C1_SCL
- R37 pad 1: +5V_USBOTG -> +3V3
- R37 pad 2: USB-VBUSDET -> AMP_MUTE0
- R38 pad 1: USB-VBUSDET -> +3V3
- R38 pad 2: GND -> AMP_FAULT0
- R39 pad 1: GND -> +3V3
- R39 pad 2: USB-ID -> AMP_PDN0
- R4 pad 1: GPIO_LED2 -> +3V3
- R4 pad 2: Net-(D2-Pad2) -> GPIO_BTN
- R40 pad 1: +3.0VA -> Net-(R40-Pad1)
- R40 pad 2: MIC-DET -> GND
- R41 pad 1: MIC-DET -> Net-(R41-Pad1)
- R41 pad 2: Net-(J5-Pad3) -> Net-(R41-Pad2)
- R42 pad 1: Net-(C46-Pad1) -> +3V3
- R42 pad 2: GNDA -> AMP_MUTE1
- R43 pad 1: Net-(C46-Pad1) -> +3V3
- R43 pad 2: Net-(R43-Pad2) -> AMP_FAULT1
- R44 pad 1: Net-(J5-Pad2) -> +3V3
- R44 pad 2: Net-(C53-Pad1) -> AMP_PDN1
- R45 pad 1: Net-(J5-Pad5) -> Net-(R41-Pad1)
- R45 pad 2: Net-(C50-Pad1) -> PCM_DOUT
- R46 pad 1: Net-(C47-Pad1) -> Net-(R46-Pad1)
- R46 pad 2: Net-(R46-Pad2) -> GND
- R47 pad 1: Net-(C50-Pad1) -> +3V3
- R47 pad 2: GNDA -> WL-SDIO-D3
- R48 pad 1: Net-(R48-Pad1) -> +3V3
- R48 pad 2: +3V3 -> WL-SDIO-D2
- R49 pad 1: Net-(R49-Pad1) -> +3V3
- R49 pad 2: +3V3 -> WL-SDIO-D1
- R50 pad 1: MIPI-SDA -> +3V3
- R50 pad 2: +3V3 -> WL-SDIO-D0
- R51 pad 1: MIPI-SCK -> +3V3
- R51 pad 2: +3V3 -> WL-SDIO-CMD
- R52 pad 1: Net-(C53-Pad1) -> +3V3
- R52 pad 2: GNDA -> WL-PMU-EN
- R54 pad 1: Net-(R54-Pad1) -> PCM_LRCLK
- R54 pad 2: BT-PCM-SYNC -> Net-(R54-Pad2)
- R58 pad 1: GNDA -> +3V3
- R58 pad 2: Net-(C63-Pad2) -> BT-WAKE-AP
- R59 pad 1: Net-(C68-Pad2) -> AP-CK32KO
- R59 pad 2: GNDA -> Net-(R59-Pad2)
- R6 pad 1: Net-(Q1-Pad1) -> GPIO_LED1
- R6 pad 2: GPIO-RST -> Net-(D2-Pad2)
- R62 pad 1: Net-(J7-Pad2) -> +3V3
- R62 pad 2: Net-(C64-Pad2) -> Net-(J1-Pad9)
- R63 pad 1: Net-(C67-Pad2) -> +3V3
- R63 pad 2: GNDA -> Net-(J1-Pad12)
- R64 pad 1: +3V3 -> Net-(R64-Pad1)
- R64 pad 2: WL-SDIO-D3 -> GND
- R65 pad 1: +3V3 -> Net-(R65-Pad1)
- R65 pad 2: WL-SDIO-D2 -> +3V3
- R66 pad 1: BT-PCM-SYNC -> EPHY_TX_P
- R66 pad 2: Net-(R66-Pad2) -> Net-(C90-Pad2)
- R67 pad 1: BT-PCM-CLK -> EPHY_TX_N
- R67 pad 2: Net-(R67-Pad2) -> Net-(C90-Pad2)
- R68 pad 1: BT-PCM-DIN -> GNDA
- R68 pad 2: Net-(R68-Pad2) -> LINE_L
- R69 pad 1: BT-PCM-DOUT -> EPHY_RX_P
- R69 pad 2: Net-(R69-Pad2) -> Net-(C93-Pad2)
- R7 pad 1: SDC0-D2 -> +3V3
- R7 pad 2: +3V3 -> Net-(D7-Pad2)
- R70 pad 1: +3V3 -> EPHY_RX_N
- R70 pad 2: WL-SDIO-D1 -> Net-(C93-Pad2)
- R71 pad 1: +3V3 -> GNDA
- R71 pad 2: WL-SDIO-D0 -> LINE_R
- R72 pad 2: WL-SDIO-CMD -> LINE_DET
- R73 pad 1: +3V3 -> Net-(C98-Pad1)
- R73 pad 2: WL-PMU-EN -> GND
- R74 pad 1: +3V3 -> GND
- R74 pad 2: BT-UART-RX -> Net-(R74-Pad2)
- R75 pad 1: +3V3 -> AP-CK32KO
- R75 pad 2: BT-WAKE-AP -> +3V3
- R76 pad 1: AP-CK32KO -> Net-(C106-Pad1)
- R76 pad 2: Net-(R76-Pad2) -> Net-(C105-Pad1)
- R77 pad 1: WL-SDIO-CLK -> Net-(C104-Pad1)
- R77 pad 2: Net-(R77-Pad2) -> +1V5
- R78 pad 1: Net-(C3-Pad1) -> +3V3
- R78 pad 2: GND -> RESETn
- R79 pad 1: Net-(C82-Pad1) -> Net-(C104-Pad1)
- R79 pad 2: VCC-DDR -> GND
- R8 pad 1: SDC0-D3 -> +3V3
- R8 pad 2: +3V3 -> I2C1_SDA
- R80 pad 1: Net-(C82-Pad1) -> Net-(R80-Pad1)
- R9 pad 1: SDC0-CMD -> SDC0_D2
- U1 pad A11: Net-(U1-PadA11) -> LCD_DCLK
- U1 pad A13: Net-(U1-PadA13) -> R3
- U1 pad A14: Net-(U1-PadA14) -> R1
- U1 pad A15: Net-(U1-PadA15) -> G4
- U1 pad A2: GPIO-RST -> GPIO_BTN
- U1 pad A3: Net-(U1-PadA3) -> Net-(R3-Pad2)
- U1 pad A5: USB-VBUSDET -> AMP_FAULT0
- U1 pad A9: Net-(U1-PadA9) -> G1
- U1 pad B1: Net-(U1-PadB1) -> SDC2_RST
- U1 pad B10: Net-(U1-PadB10) -> LCD_VSYNC
- U1 pad B11: Net-(U1-PadB11) -> LCD_ENAB
- U1 pad B12: Net-(U1-PadB12) -> R4
- U1 pad B13: Net-(U1-PadB13) -> R2
- U1 pad B14: Net-(U1-PadB14) -> R0
- U1 pad B15: Net-(U1-PadB15) -> G5
- U1 pad B16: Net-(U1-PadB16) -> B4
- U1 pad B2: Net-(U1-PadB2) -> SDC2_CMD
- U1 pad B5: MIC-DET -> AMP_FAULT1
- U1 pad B9: Net-(U1-PadB9) -> G0
- U1 pad C1: Net-(U1-PadC1) -> SDC2_D3
- U1 pad C10: Net-(U1-PadC10) -> LCD_HSYNC
- U1 pad C11: Net-(U1-PadC11) -> B1
- U1 pad C12: Net-(U1-PadC12) -> R5
- U1 pad C13: Net-(R2-Pad1) -> Net-(R12-Pad1)
- U1 pad C15: Net-(U1-PadC15) -> G2
- U1 pad C16: Net-(U1-PadC16) -> B5
- U1 pad C2: Net-(U1-PadC2) -> SDC2_D0
- U1 pad C3: Net-(U1-PadC3) -> SDC2_D4
- U1 pad C7: GPIO_LED1 -> LINE_DET
- U1 pad C8: GPIO_LED2 -> LCD_PWM
- U1 pad D1: Net-(U1-PadD1) -> SDC2_D7
- U1 pad D2: Net-(U1-PadD2) -> SDC2_D6
- U1 pad D3: Net-(U1-PadD3) -> SDC2_D5
- U1 pad E13: Net-(U1-PadE13) -> AMP_MUTE0
- U1 pad F14: Net-(U1-PadF14) -> GPIO_LED0
- U1 pad F3: Net-(U1-PadF3) -> SDC2_D1
- U1 pad F4: Net-(U1-PadF4) -> SDC2_D2
- U1 pad F5: Net-(R83-Pad1) -> Net-(R81-Pad1)
- U1 pad F6: VCC-DDR -> +1V5
- U1 pad F7: VCC-DDR -> +1V5
- U1 pad F8: VCC-DDR -> +1V5
- U1 pad G13: Net-(U1-PadG13) -> GPIO_LED1
- U1 pad G15: Net-(U1-PadG15) -> AMP_PDN0
- U1 pad G16: MIPI-SCK -> I2C1_SCL
- U1 pad G8: VCC-DDR -> +1V5
- U1 pad H13: Net-(U1-PadH13) -> AMP_PDN1
- U1 pad H6: Net-(C82-Pad1) -> Net-(C104-Pad1)
- U1 pad H8: VCC-DDR -> +1V5
- U1 pad J13: Net-(U1-PadJ13) -> AMP_MUTE1
- U1 pad J14: Net-(U1-PadJ14) -> B2
- U1 pad J15: Net-(U1-PadJ15) -> B3
- U1 pad J16: MIPI-SDA -> I2C1_SDA
- U1 pad J5: Net-(R82-Pad1) -> Net-(R80-Pad1)
- U1 pad J8: VCC-DDR -> +1V5
- U1 pad K15: Net-(U1-PadK15) -> B0
- U1 pad L15: Net-(U1-PadL15) -> G3
- U1 pad M1: SDC0-DET# -> SDC0_DET#
- U1 pad M13: BT-PCM-DIN -> PCM_DIN
- U1 pad M2: SDC0-D2 -> SDC0_D2
- U1 pad M6: Net-(R34-Pad1) -> Net-(R25-Pad1)
- U1 pad M9: Net-(C85-Pad1) -> Net-(C102-Pad1)
- U1 pad N10: Net-(C3-Pad1) -> Net-(C98-Pad1)
- U1 pad N2: SDC0-CMD -> SDC0_CMD
- U1 pad N3: SDC0-D3 -> SDC0_D3
- U1 pad N6: +3.3V_RTC -> +3V3
- U1 pad P1: SDC0-D0 -> SDC0_D0
- U1 pad P14: BT-PCM-CLK -> PCM_BCLK
- U1 pad P2: SDC0-CLK -> SDC0_CLK
- U1 pad P4: Net-(C94-Pad1) -> Net-(C113-Pad1)
- U1 pad P6: Net-(R89-Pad2) -> Net-(R74-Pad2)
- U1 pad R1: SDC0-D1 -> SDC0_D1
- U1 pad R12: Net-(U1-PadR12) -> LINE_L
- U1 pad R13: Net-(R81-Pad1) -> Net-(R64-Pad1)
- U1 pad R3: Net-(C97-Pad1) -> Net-(C106-Pad1)
- U1 pad R4: Net-(C93-Pad1) -> Net-(C109-Pad1)
- U1 pad R7: NMI -> Net-(R65-Pad1)
- U1 pad T12: Net-(U1-PadT12) -> LINE_R
- U1 pad T14: BT-PCM-SYNC -> PCM_LRCLK
- U1 pad T15: BT-PCM-DOUT -> PCM_DOUT
- U1 pad T3: Net-(C96-Pad1) -> Net-(C105-Pad1)
- U1 pad T5: Net-(C90-Pad1) -> Net-(C107-Pad1)
- U3 pad 1: MIPI-SDA -> +3V3
- U3 pad 2: MIPI-SCK -> GND
- U3 pad 3: Net-(U3-Pad3) -> Net-(L2-Pad1)
- U3 pad 4: Net-(Q1-Pad3) -> +3V3
- U3 pad 5: Net-(U3-Pad5) -> Net-(R16-Pad2)
- U4 pad 1: +3.0VA -> Net-(C7-Pad2)
- U4 pad 2: GND -> VBUS
- U4 pad 3: Net-(L3-Pad1) -> Net-(C7-Pad1)
- U4 pad 4: IPS -> GND
- U4 pad 5: Net-(R30-Pad2) -> Net-(R18-Pad2)
- U5 pad 1: +5V_USBOTG -> +3V3
- U5 pad 3: Net-(R36-Pad1) -> Net-(L3-Pad1)
- U5 pad 4: USB-DRV -> +3V3
- U5 pad 5: +5V -> Net-(R23-Pad2)
- U6 pad 1: Net-(C51-Pad1) -> +3V3
- U6 pad 2: Net-(C52-Pad1) -> GND
- U6 pad 4: GND -> Net-(U6-Pad4)
- U7 pad 1: GND -> Net-(D5-Pad2)
- U7 pad 10: Net-(U7-Pad10) -> GND
- U7 pad 12: WL-PMU-EN -> Net-(R34-Pad2)
- U7 pad 13: WL-WAKE-AP -> Net-(R33-Pad2)
- U7 pad 14: WL-SDIO-D2 -> Net-(U7-Pad14)
- U7 pad 15: WL-SDIO-D3 -> Net-(U7-Pad15)
- U7 pad 16: WL-SDIO-CMD -> Net-(R29-Pad1)
- U7 pad 17: Net-(R77-Pad2) -> Net-(U7-Pad17)
- U7 pad 18: WL-SDIO-D0 -> Net-(R28-Pad1)
- U7 pad 19: WL-SDIO-D1 -> Net-(U7-Pad19)
- U7 pad 2: Net-(C78-Pad2) -> Net-(D5-Pad2)
- U7 pad 20: GND -> Net-(U7-Pad20)
- U7 pad 21: Net-(L4-Pad2) -> Net-(C40-Pad2)
- U7 pad 22: +3V3 -> GND
- U7 pad 23: Net-(C48-Pad1) -> Net-(C41-Pad2)
- U7 pad 24: Net-(R76-Pad2) -> Net-(C38-Pad2)
- U7 pad 25: Net-(R69-Pad2) -> GND
- U7 pad 4: Net-(U7-Pad4) -> Net-(D5-Pad1)
- U7 pad 5: Net-(U7-Pad5) -> Net-(D5-Pad1)
- U7 pad 6: AP-WAKE-BT -> Net-(R35-Pad1)
- U7 pad 7: BT-WAKE-AP -> I2C1_SCL
- U7 pad 8: Net-(U7-Pad8) -> I2C1_SDA
- U7 pad 9: +3V3 -> Net-(R30-Pad1)
- Y1 pad 1: Net-(C52-Pad1) -> Net-(C105-Pad1)
- Y1 pad 2: GND -> Net-(C106-Pad1)
- Y2 pad 1: Net-(C96-Pad1) -> Net-(C109-Pad1)
- Y2 pad 2: Net-(C97-Pad1) -> GND
- Y3 pad 1: Net-(C93-Pad1) -> Net-(C118-Pad1)
- Y3 pad 3: Net-(C94-Pad1) -> Net-(C117-Pad1)
Routing:
- net VBUS: track 0.00 -> 234.7 mm
- net GND: track 231.0 -> 35.2 mm, vias 211 -> 225
- net I2C1_SCL: track 0.00 -> 123.0 mm, vias 0 -> 7
- net I2C1_SDA: track 0.00 -> 118.5 mm, vias 0 -> 7
- net Net-(C70-Pad2): track 0.00 -> 116.1 mm, vias 0 -> 8
- net IPS: track 106.5 -> 0.00 mm, vias 19 -> 0
- net +3V3: track 171.6 -> 70.3 mm, vias 25 -> 3
- net +3.0VA: track 112.4 -> 12.7 mm, vias 15 -> 2
- net Net-(C72-Pad1): track 0.00 -> 98.7 mm, vias 0 -> 8
- net AMP_FAULT1: track 0.00 -> 81.7 mm, vias 0 -> 4
- net PCM_BCLK: track 0.00 -> 76.2 mm, vias 0 -> 4
- net PCM_LRCLK: track 0.00 -> 75.8 mm, vias 0 -> 4
- net Net-(C51-Pad2): track 0.00 -> 75.3 mm, vias 0 -> 8
- net AMP_PDN1: track 0.00 -> 72.8 mm, vias 0 -> 4
- net AMP_MUTE1: track 0.00 -> 72.4 mm, vias 0 -> 4
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- added copper zone on F.Cu, net Net-(C50-Pad1)
- added copper zone on F.Cu, net Net-(C52-Pad1)
- added copper zone on F.Cu, net Net-(C56-Pad1)
- added copper zone on F.Cu, net Net-(C60-Pad1)
- added copper zone on F.Cu, net Net-(C69-Pad1)
- added copper zone on F.Cu, net Net-(C71-Pad1)
- added copper zone on F.Cu, net Net-(C75-Pad1)
- added copper zone on F.Cu, net Net-(C79-Pad1)
- added copper zone on F.Cu, net VBUS
- removed copper zone on F.Cu, net +1.1V
- removed copper zone on In1.Cu, net +1.1V
- removed copper zone on In2.Cu, net +1.1V
- removed copper zone on B.Cu, net +3V3
- removed copper zone on F.Cu, net +3V3
- removed copper zone on In1.Cu, net +3V3
- removed copper zone on B.Cu, net +5V
- removed copper zone on In2.Cu, net GND
- removed copper zone on In1.Cu, net GNDA
- removed copper zone on F.Cu, net IPS
- removed copper zone on In1.Cu, net IPS
- removed copper zone on F.Cu, net VCC-DDR
- removed copper zone on In1.Cu, net VCC-DDR
Other:
- board size 50 x 49.3 mm -> 96 x 100 mm
- net class DC added: clearance 0.2, trace_width 0.127, via_dia 0.6, via_drill 0.3
- net class HV added: clearance 0.5, trace_width 0.127, via_dia 0.6, via_drill 0.3
- board text removed: "CFG"

Commit message: layout final?
Parts:
- removed C114: 100n 50V, otter:C_0603
- removed C121, C122, C24, C30, C32, C33, C34: 100n, otter:C_0402
- removed C14, C15, C25, C26, C27, C28, C99: 10u, otter:C_0603
- added C110: 100n, otter:C_0402, F.Cu at (175.2, 137.2)
- added C112: 470n 25V, otter:C_0603, F.Cu at (189.4, 136.7)
- added D8: ESD5302F, Package_TO_SOT_SMD:SOT-23, F.Cu at (183.8, 57.1)
- added G***: LOGO, ottercast:ottercast_mask, F.Cu at (160.0, 131.0)
- added G***: LOGO, ottercast:ottercast_enig, F.Cu at (160.0, 131.0)
- added G***: LOGO, ottercast:ottercast_silk, F.Cu at (160.0, 131.0)
- added J7: AFA07-S10FCC-00, Connector_FFC-FPC:TE_1-84952-0_1x10-1MP_P1.0mm_Horizontal, F.Cu at (179.4, 115.3)
- added JP10: JMP, Jumper:SolderJumper-2_P1.3mm_Bridged_Pad1.0x1.5mm, B.Cu at (171.8, 143.5)
- added JP11: GNDA, Jumper:SolderJumper-2_P1.3mm_Bridged_Pad1.0x1.5mm, B.Cu at (188.8, 88.5)
- added JP9: JMP, Jumper:SolderJumper-2_P1.3mm_Bridged_Pad1.0x1.5mm, B.Cu at (171.8, 141.5)
- added R60: 0R, otter:R_0402, F.Cu at (155.9, 102.7)
- added R61: 47k, otter:R_0402, F.Cu at (175.2, 135.6)
- added R82: 47k, otter:R_0402, F.Cu at (189.1, 137.7)
- added R83: 10R, otter:R_0402, F.Cu at (184.2, 137.2)
- added R84: 2.2k, otter:R_0402, F.Cu at (177.9, 111.2)
- added R85: 2.2k, otter:R_0402, F.Cu at (177.9, 110.3)
- added U8: AP3019A, Package_TO_SOT_SMD:SOT-23-6, F.Cu at (186.4, 136.8)
- 3V3 PG: renamed from D7
- C29, J10: moved to B.Cu
- C85: value 10p -> 18p
- C86, C87: value 1p -> DNP
- L12: value 2.2nH -> 22u; footprint otter:L_0402 -> otter:Inductor_4040
- R31, R32: value DNP -> 0R
- SW1: footprint Button_Switch_THT:SW_Tactile_SPST_Angled_PTS645Vx58-2LFS -> Button_Switch_SMD:SW_SPST_EVQP7C; moved to B.Cu
- moved C86 86.7 mm to (155.4, 103.8)
- moved C31 80.0 mm to (155.0, 84.5), turned to 180 degrees
- moved C20 71.8 mm to (160.3, 83.2)
- moved C12 70.6 mm to (169.1, 83.2)
- moved SW1 69.9 mm to (157.6, 51.5)
- moved C19 68.0 mm to (168.7, 90.5), turned to 90 degrees
- moved C11 67.7 mm to (171.4, 84.5), turned to 90 degrees
- moved C13 67.3 mm to (166.7, 83.2), turned to 180 degrees
- moved R57 64.4 mm to (159.3, 100.2), turned to 90 degrees
- moved C29 62.9 mm to (173.9, 93.3), turned to 315 degrees
- moved C87 58.8 mm to (155.4, 101.5)
- moved C85 53.5 mm to (155.9, 100.2), turned to 90 degrees
- moved C82 51.8 mm to (162.2, 100.2), turned to 270 degrees
- moved C35 50.8 mm to (183.0, 93.7), turned to 90 degrees
- moved C16 47.3 mm to (171.8, 59.8), turned to 270 degrees
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Connections:
- net UART0_TX renamed Net-(U1-PadB6)
- J10 pad 1: Net-(J10-Pad1) -> GND
- J10 pad 10: B2 -> R4
- J10 pad 11: B3 -> R3
- J10 pad 12: B4 -> R2
- J10 pad 13: B5 -> R1
- J10 pad 14: G0 -> G5
- J10 pad 15: G1 -> G4
- J10 pad 16: G2 -> G3
- J10 pad 17: G3 -> G2
- J10 pad 18: G4 -> G1
- J10 pad 19: G5 -> G0
- J10 pad 2: Net-(J10-Pad2) -> +3V3
- J10 pad 20: R0 -> B5
- J10 pad 21: R1 -> B4
- J10 pad 22: R2 -> B3
- J10 pad 23: R3 -> B2
- J10 pad 24: R4 -> B1
- J10 pad 25: R5 -> LCD_ENAB
- J10 pad 27: LCD_ENAB -> LCD_HSYNC
- J10 pad 28: LCD_HSYNC -> LCD_VSYNC
- J10 pad 29: LCD_VSYNC -> LEDA
- J10 pad 3: Net-(J10-Pad3) -> +3V3
- J10 pad 30: Net-(J10-Pad30) -> LEDK
- J10 pad 8: B0 -> LCD_RESET
- J10 pad 9: B1 -> R5
- L12 pad 1: Net-(AE1-Pad1) -> +3V3
- L12 pad 2: Net-(C85-Pad1) -> Net-(L12-Pad2)
- U1 pad C6: UART0_RX -> I2C0_INT
Routing:
- net +3V3: track 70.3 -> 297.1 mm, vias 3 -> 38
- net GPIO_BTN: track 0.45 -> 106.9 mm, vias 1 -> 4
- net GND: track 35.2 -> 104.3 mm, vias 225 -> 430
- net LINE_DET: track 0.34 -> 68.2 mm, vias 1 -> 3
- net G0: track 2.28 -> 59.2 mm
- net B2: track 3.52 -> 60.1 mm, vias 1 -> 4
- net G1: track 1.87 -> 58.0 mm
- net B3: track 2.20 -> 57.7 mm, vias 1 -> 4
- net G3: track 3.48 -> 57.8 mm, vias 1 -> 2
- net LCD_HSYNC: track 2.88 -> 55.9 mm, vias 1 -> 3
- net LCD_ENAB: track 2.16 -> 54.1 mm, vias 1 -> 3
- net B4: track 2.33 -> 53.5 mm, vias 1 -> 3
- net G2: track 3.30 -> 54.3 mm, vias 1 -> 3
- net G4: track 1.60 -> 52.0 mm, vias 1 -> 3
- net R1: track 1.52 -> 51.5 mm, vias 1 -> 3
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- added copper zone on In1.Cu, net +1.1V
- added copper zone on In1.Cu, net +1V5
- added copper zone on In1.Cu, net +3V3
- added copper zone on In1.Cu, net GND
- added copper zone on In2.Cu, net GND
Other:
- board text added: "FRONT"
- board text added: "GND SCL SDA INT 3V3 LED1 LED0 BTN 3V3 GND"
- board text added: "GND TXD RXD"
- board text added: "LCD"
- board text added: "LED0"
- board text added: "LED1"

Commit message: V1.0 order release
Parts:
- D7: renamed from 3V3 PG
- R18: value 31.25k -> 47k
- R21: value 10k -> 15k
- R24: value 68k -> 100k
- R54, R55, R56: value DNP -> 100R
- R75: value 5k1 -> 5.6k
- R77, R79: value 2k2 -> 2.2k
- R82: value 47k -> 10k
- moved G*** 0.71 mm to (159.5, 131.5) (x3)
- moved R41 0.20 mm to (134.3, 90.0)
- moved C47 0.10 mm to (134.3, 92.1)
- moved R40 0.10 mm to (134.3, 91.3)
Connections:
- C43 pad 2: Net-(C43-Pad2) -> +3V3
- C44 pad 2: Net-(C43-Pad2) -> +3V3
- C62 pad 2: Net-(C62-Pad2) -> +3V3
- C63 pad 2: Net-(C62-Pad2) -> +3V3
- U10 pad 6: Net-(C62-Pad2) -> +3V3
- U9 pad 6: Net-(C43-Pad2) -> +3V3
Routing:
- net +3V3: track 297.1 -> 355.1 mm, vias 38 -> 40
- net Net-(C62-Pad2): track 4.02 -> 0.00 mm
- net Net-(C43-Pad2): track 4.02 -> 0.00 mm
Other:
- board text added: "Hardware: @JanHenrikH, @FauthNiklas Software: @Manawyrm, @Toble_Miner Rev 1.1"
- board text added: "OtterCast Amp"

Commit message: V1.2 production release
Parts:
- removed JP10, JP9: JMP, Jumper:SolderJumper-2_P1.3mm_Bridged_Pad1.0x1.5mm
- added B1: TestPoint, TestPoint:TestPoint_Pad_1.0x1.0mm, F.Cu at (181.6, 134.9)
- added COPI: TestPoint, TestPoint:TestPoint_Pad_1.0x1.0mm, F.Cu at (188.2, 143.9)
- added CS: TestPoint, TestPoint:TestPoint_Pad_1.0x1.0mm, F.Cu at (188.2, 142.5)
- added DCLK: TestPoint, TestPoint:TestPoint_Pad_1.0x1.0mm, F.Cu at (181.6, 136.3)
- added ENAB: TestPoint, TestPoint:TestPoint_Pad_1.0x1.0mm, F.Cu at (181.6, 137.7)
- added HSYNC: TestPoint, TestPoint:TestPoint_Pad_1.0x1.0mm, F.Cu at (183.0, 137.7)
- added R86: 0R, otter:R_0402, F.Cu at (189.3, 131.6)
- added R87: 0R, otter:R_0402, F.Cu at (190.2, 131.6)
- added R88: 0R, otter:R_0402, F.Cu at (191.1, 131.6)
- added R89: 2.2k, otter:R_0402, F.Cu at (171.4, 82.8)
- added SCLK: TestPoint, TestPoint:TestPoint_Pad_1.0x1.0mm, F.Cu at (188.2, 141.1)
- added VSYNC: TestPoint, TestPoint:TestPoint_Pad_1.0x1.0mm, F.Cu at (183.0, 136.3)
- 3V3 PG: renamed from D7
- C117, C118: value 18p -> 22pF
- Q1: value IRF8736 -> DMP4015SS
- moved R62 1.75 mm to (168.9, 58.1)
- moved R63 1.73 mm to (168.9, 59.0)
- moved J10 1.20 mm to (180.9, 142.7)
- moved R8 0.28 mm to (171.4, 81.1)
- moved R36 0.26 mm to (170.5, 81.1)
Connections:
- J1 pad 10: EPHY_LINK_LED -> GND
- J1 pad 11: EPHY_SPD_LED -> GND
- J10 pad 5: Net-(J10-Pad5) -> LCD_SDA
- J10 pad 6: Net-(J10-Pad6) -> LCD_SCL
- J10 pad 7: Net-(J10-Pad7) -> LCD_CS
- R62 pad 1: +3V3 -> EPHY_LINK_LED
- R63 pad 1: +3V3 -> EPHY_SPD_LED
- U1 pad R14: USB-ID -> I2C1_INT
- U7 pad 19: Net-(U7-Pad19) -> I2C1_INT
Routing:
- net I2C1_INT: track 0.00 -> 28.3 mm, vias 0 -> 2
- net LCD_CS: track 0.00 -> 26.4 mm, vias 0 -> 3
- net LCD_SCL: track 0.00 -> 25.9 mm, vias 0 -> 3
- net LCD_SDA: track 0.00 -> 25.7 mm, vias 0 -> 3
- net I2C0_SDA: track 21.5 -> 46.4 mm, vias 2 -> 3
- net I2C0_SCL: track 21.7 -> 46.4 mm, vias 2 -> 3
- net I2C0_INT: track 22.0 -> 46.5 mm, vias 3 -> 4
- net EPHY_SPD_LED: track 55.2 -> 38.5 mm, vias 1 -> 2
- net EPHY_LINK_LED: track 45.8 -> 39.3 mm, vias 1 -> 2
- net Net-(J10-Pad7): track 5.17 -> 0.00 mm
- net Net-(J10-Pad6): track 4.34 -> 0.00 mm
- net Net-(J1-Pad9): track 7.40 -> 5.51 mm
- net Net-(J1-Pad12): track 21.0 -> 19.4 mm
- net LCD_ENAB: track 54.1 -> 55.6 mm
- net LCD_HSYNC: track 55.9 -> 57.2 mm
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Other:
- outline, holes or cut-outs redrawn
- board text added: "FRONT EXPANSION"
- board text added: "Hardware: @JanHenrikH, @FauthNiklas Software: @Manawyrm, @Toble_Miner Rev 1.2"
- board text added: "POWER"
- board text added: "STATUS"
- board text removed: "FRONT"
- board text removed: "Hardware: @JanHenrikH, @FauthNiklas Software: @Manawyrm, @Toble_Miner Rev 1.1"
- board text removed: "LED0"
- board text removed: "LED1"
