File: lcd.sch (KiCad schematic (older format))
At the start: 1 part, among them J10 FH26W-33S-0.3SHW

Commit message: layout final?
Parts:
- added C110: 100n, otter:C_0402, symbol Device:C_Small
- added C112: 470n 25V, otter:C_0603, symbol Device:C_Small
- added J7: AFA07-S10FCC-00, Connector_FFC-FPC:TE_1-84952-0_1x10-1MP_P1.0mm_Horizontal, symbol Connector_Generic_MountingPin:Conn_01x10_MountingPin
- added JP10, JP9: JMP, Jumper:SolderJumper-2_P1.3mm_Bridged_Pad1.0x1.5mm, symbol Device:Jumper_NC_Small
- added L12: 22u, otter:Inductor_4040, symbol Device:L_Small
- added R61, R82: 47k, otter:R_0402, symbol Device:R_Small
- added R83: 10R, otter:R_0402, symbol Device:R_Small
- added R84, R85: 2.2k, otter:R_0402, symbol Device:R_Small
- added U8: AP3019A, Package_TO_SOT_SMD:SOT-23-6, symbol otter:AP3019A
Connections:
- net B0: no longer J10.8 (Pin_8)
- net B1: now also J10.24 (Pin_24); no longer J10.9 (Pin_9)
- net B2: now also J10.23 (Pin_23); no longer J10.10 (Pin_10)
- net B3: now also J10.22 (Pin_22); no longer J10.11 (Pin_11)
- net B4: now also J10.21 (Pin_21); no longer J10.12 (Pin_12)
- net B5: now also J10.20 (Pin_20); no longer J10.13 (Pin_13)
- net G0: now also J10.19 (Pin_19); no longer J10.14 (Pin_14)
- net G1: now also J10.18 (Pin_18); no longer J10.15 (Pin_15)
- net G2: now also J10.17 (Pin_17); no longer J10.16 (Pin_16)
- net G3: now also J10.16 (Pin_16); no longer J10.17 (Pin_17)
- net G4: now also J10.15 (Pin_15); no longer J10.18 (Pin_18)
- net G5: now also J10.14 (Pin_14); no longer J10.19 (Pin_19)
- net GND: now also J10.1 (Pin_1), C110.2, C112.1, J7.1 (Pin_1), J7.10 (Pin_10), J7.MP (MountPin), JP10.1, JP9.1, R83.2, U8.2 (GND)
- net LCD_ENAB: now also J10.25 (Pin_25); no longer J10.27 (Pin_27)
- net LCD_HSYNC: now also J10.27 (Pin_27); no longer J10.28 (Pin_28)
- net LCD_PWM: now also R82.2, U8.4 (EN)
- net LCD_VSYNC: now also J10.28 (Pin_28); no longer J10.29 (Pin_29)
- net R0: no longer J10.20 (Pin_20)
- net R1: now also J10.13 (Pin_13); no longer J10.21 (Pin_21)
- net R2: now also J10.12 (Pin_12); no longer J10.22 (Pin_22)
- net R3: now also J10.11 (Pin_11); no longer J10.23 (Pin_23)
- net R4: now also J10.10 (Pin_10); no longer J10.24 (Pin_24)
- net R5: now also J10.9 (Pin_9); no longer J10.25 (Pin_25)
- net +3V3: now reaches J10.2 (Pin_2)
- net +3V3: now also J10.3 (Pin_3), J7.5 (Pin_5), J7.9 (Pin_9), L12.1, R61.1, R82.1, R84.1, R85.1, U8.6 (IN)
- net LEDK: now reaches J10.30 (Pin_30)
- net LEDK: now also R83.1, U8.3 (FB)
- net at J10.6 (Pin_6): now also JP9.2
- net at J10.7 (Pin_7): now also JP10.2
- new net: L12.2, U8.1 (SW)
- new net GPIO_BTN: J7.8 (Pin_8)
- new net GPIO_LED0: J7.7 (Pin_7)
- new net GPIO_LED1: J7.6 (Pin_6)
- new net I2C0_INT: J7.4 (Pin_4)
- new net I2C0_SCL: J7.2 (Pin_2), R85.2
- new net I2C0_SDA: J7.3 (Pin_3), R84.2
- new net LCD_RESET: C110.1, J10.8 (Pin_8), R61.2
- new net LEDA: C112.2, J10.29 (Pin_29), U8.5 (OUT)
- no-connect marks 0 -> 5
Other:
- moved on the sheet: J10

Commit message: V1.0 order release
Parts:
- R82: value 47k -> 10k
Other:
- moved on the sheet: C110, J7, R61
Changed lines of the file:
@@
 Comment4 ""
 $EndDescr
-Text GLabel 5150 2050 0    50   Input ~ 0
+Text GLabel 5200 2100 0    50   Input ~ 0
 B0
 Text GLabel 7550 3250 0    50   Input ~ 0
@@
 Text GLabel 7550 2250 0    50   Input ~ 0
 G5
-Text GLabel 5150 2150 0    50   Input ~ 0
+Text GLabel 5200 2200 0    50   Input ~ 0
 R0
 Text GLabel 7550 2150 0    50   Input ~ 0
@@
 Text GLabel 7550 1650 0    50   Input ~ 0
 LCD_RESET
-Text GLabel 5400 1600 0    50   Input ~ 0
+Text GLabel 5450 1650 0    50   Input ~ 0
 LCD_RESET
 Text GLabel 7550 2850 0    50   Input ~ 0
@@
 P 3000 2350
 F 0 "R82" H 3059 2396 50  0000 L CNN
-F 1 "47k" H 3059 2305 50  0000 L CNN
+F 1 "10k" H 3059 2305 50  0000 L CNN
 F 2 "otter:R_0402" H 3000 2350 50  0001 C CNN
 F 3 "~" H 3000 2350 50  0001 C CNN
@@
 L Device:R_Small R61
 U 1 1 60C8D955
-P 5450 1450
-F 0 "R61" H 5509 1496 50  0000 L CNN
-F 1 "47k" H 5509 1405 50  0000 L CNN
-F 2 "otter:R_0402" H 5450 1450 50  0001 C CNN
-F 3 "~" H 5450 1450 50  0001 C CNN
-	1    5450 1450
+P 5500 1500
+F 0 "R61" H 5559 1546 50  0000 L CNN
+F 1 "47k" H 5559 1455 50  0000 L CNN
+F 2 "otter:R_0402" H 5500 1500 50  0001 C CNN
+F 3 "~" H 5500 1500 50  0001 C CNN
+	1    5500 1500
 	1    0    0    -1
 $EndComp
@@
 L power:+3V3 #PWR0242
 U 1 1 60C8DD76
-P 5450 1350
-F 0 "#PWR0242" H 5450 1200 50  0001 C CNN
-F 1 "+3V3" H 5465 1523 50  0000 C CNN
-F 2 "" H 5450 1350 50  0001 C CNN
-F 3 "" H 5450 1350 50  0001 C CNN
-	1    5450 1350
+P 5500 1400
+F 0 "#PWR0242" H 5500 1250 50  0001 C CNN
+F 1 "+3V3" H 5515 1573 50  0000 C CNN
+F 2 "" H 5500 1400 50  0001 C CNN
+F 3 "" H 5500 1400 50  0001 C CNN
+	1    5500 1400
 	1    0    0    -1
 $EndComp
@@
 L Device:C_Small C110
 U 1 1 60C8E672
-P 5450 1750
-F 0 "C110" H 5542 1796 50  0000 L CNN
-F 1 "100n" H 5542 1705 50  0000 L CNN
-F 2 "otter:C_0402" H 5450 1750 50  0001 C CNN
-F 3 "~" H 5450 1750 50  0001 C CNN
-	1    5450 1750
+P 5500 1800
+F 0 "C110" H 5592 1846 50  0000 L CNN
+F 1 "100n" H 5592 1755 50  0000 L CNN
+F 2 "otter:C_0402" H 5500 1800 50  0001 C CNN
+F 3 "~" H 5500 1800 50  0001 C CNN
+	1    5500 1800
 	1    0    0    -1
 $EndComp
@@
 L otter:GND #PWR0243
 U 1 1 60C8ED81
-P 5450 1850
-F 0 "#PWR0243" H 5450 1600 50  0001 C CNN
-F 1 "GND" H 5455 1677 50  0000 C CNN
-F 2 "" H 5450 1850 60  0000 C CNN
-F 3 "" H 5450 1850 60  0000 C CNN
-	1    5450 1850
-	1    0    0    -1
-$EndComp
-Wire Wire Line
-	5450 1650 5450 1600
-Wire Wire Line
-	5400 1600 5450 1600
-Connection ~ 5450 1600
-Wire Wire Line
-	5450 1600 5450 1550
+P 5500 1900
+F 0 "#PWR0243" H 5500 1650 50  0001 C CNN
+F 1 "GND" H 5505 1727 50  0000 C CNN
+F 2 "" H 5500 1900 60  0000 C CNN
+F 3 "" H 5500 1900 60  0000 C CNN
+	1    5500 1900
+	1    0    0    -1
+$EndComp
+Wire Wire Line
+	5500 1700 5500 1650
+Wire Wire Line
+	5450 1650 5500 1650
+Connection ~ 5500 1650
+Wire Wire Line
+	5500 1650 5500 1600
 $Comp
 L Connector_Generic_MountingPin:Conn_01x10_MountingPin J7
 U 1 1 60C92491
-P 5450 3750
-F 0 "J7" H 5538 3664 50  0000 L CNN
-F 1 "AFA07-S10FCC-00" H 5538 3573 50  0000 L CNN
-F 2 "Connector_FFC-FPC:TE_1-84952-0_1x10-1MP_P1.0mm_Horizontal" H 5450 3750 50  0001 C CNN
-F 3 "~" H 5450 3750 50  0001 C CNN
-	1    5450 3750
+P 5500 3650
+F 0 "J7" H 5588 3564 50  0000 L CNN
+F 1 "AFA07-S10FCC-00" H 5588 3473 50  0000 L CNN
+F 2 "Connector_FFC-FPC:TE_1-84952-0_1x10-1MP_P1.0mm_Horizontal" H 5500 3650 50  0001 C CNN
+F 3 "~" H 5500 3650 50  0001 C CNN
+	1    5500 3650
 	1    0    0    -1
 $EndComp
@@
 L otter:GND #PWR0244
 U 1 1 60C92F25
-P 5450 4450
-F 0 "#PWR0244" H 5450 4200 50  0001 C CNN
-F 1 "GND" H 5455 4277 50  0000 C CNN
-F 2 "" H 5450 4450 60  0000 C CNN
-F 3 "" H 5450 4450 60  0000 C CNN
-	1    5450 4450
+P 5500 4350
+F 0 "#PWR0244" H 5500 4100 50  0001 C CNN
+F 1 "GND" H 5505 4177 50  0000 C CNN
+F 2 "" H 5500 4350 60  0000 C CNN
+F 3 "" H 5500 4350 60  0000 C CNN
+	1    5500 4350
 	1    0    0    -1
 $EndComp
@@
 L otter:GND #PWR0245
 U 1 1 60C94CDF
-P 5250 4250
-F 0 "#PWR0245" H 5250 4000 50  0001 C CNN
-F 1 "GND" V 5250 4100 50  0000 R CNN
-F 2 "" H 5250 4250 60  0000 C CNN
-F 3 "" H 5250 4250 60  0000 C CNN
-	1    5250 4250
+P 5300 4150
+F 0 "#PWR0245" H 5300 3900 50  0001 C CNN
+F 1 "GND" V 5300 4000 50  0000 R CNN
+F 2 "" H 5300 4150 60  0000 C CNN
+F 3 "" H 5300 4150 60  0000 C CNN
+	1    5300 4150
 	0    1    -1   0
 $EndComp
@@
 L otter:GND #PWR0246
 U 1 1 60C950B3
-P 5250 3350
-F 0 "#PWR0246" H 5250 3100 50  0001 C CNN
-F 1 "GND" V 5250 3200 50  0000 R CNN
-F 2 "" H 5250 3350 60  0000 C CNN
-F 3 "" H 5250 3350 60  0000 C CNN
-	1    5250 3350
+P 5300 3250
+F 0 "#PWR0246" H 5300 3000 50  0001 C CNN
+F 1 "GND" V 5300 3100 50  0000 R CNN
+F 2 "" H 5300 3250 60  0000 C CNN
+F 3 "" H 5300 3250 60  0000 C CNN
+	1    5300 3250
 	0    1    -1   0
 $EndComp
-Text GLabel 5250 3450 0    50   Input ~ 0
+Text GLabel 5300 3350 0    50   Input ~ 0
 I2C0_SCL
-Text GLabel 5250 3550 0    50   Input ~ 0
+Text GLabel 5300 3450 0    50   Input ~ 0
 I2C0_SDA
-Text GLabel 5250 3950 0    50   Input ~ 0
+Text GLabel 5300 3850 0    50   Input ~ 0
 GPIO_LED0
-Text GLabel 5250 3850 0    50   Input ~ 0
+Text GLabel 5300 3750 0    50   Input ~ 0
 GPIO_LED1
-Text GLabel 5250 4050 0    50   Input ~ 0
+Text GLabel 5300 3950 0    50   Input ~ 0
 GPIO_BTN
 $Comp
@@
 Text GLabel 3900 3800 3    50   Input ~ 0
 I2C0_SDA
-Text GLabel 5250 3650 0    50   Input ~ 0
+Text GLabel 5300 3550 0    50   Input ~ 0
 I2C0_INT
 $Comp
 L power:+3V3 #PWR0249
 U 1 1 60D0E470
-P 5250 4150
-F 0 "#PWR0249" H 5250 4000 50  0001 C CNN
-F 1 "+3V3" V 5250 4300 50  0000 L CNN
-F 2 "" H 5250 4150 50  0001 C CNN
-F 3 "" H 5250 4150 50  0001 C CNN
-	1    5250 4150
+P 5300 4050
+F 0 "#PWR0249" H 5300 3900 50  0001 C CNN
+F 1 "+3V3" V 5300 4200 50  0000 L CNN
+F 2 "" H 5300 4050 50  0001 C CNN
+F 3 "" H 5300 4050 50  0001 C CNN
+	1    5300 4050
 	0    -1   1    0
 $EndComp
@@
 L power:+3V3 #PWR0250
 U 1 1 60D0F072
-P 5250 3750
-F 0 "#PWR0250" H 5250 3600 50  0001 C CNN
-F 1 "+3V3" V 5250 3900 50  0000 L CNN
-F 2 "" H 5250 3750 50  0001 C CNN
-F 3 "" H 5250 3750 50  0001 C CNN
-	1    5250 3750
+P 5300 3650
+F 0 "#PWR0250" H 5300 3500 50  0001 C CNN
+F 1 "+3V3" V 5300 3800 50  0000 L CNN
+F 2 "" H 5300 3650 50  0001 C CNN
+F 3 "" H 5300 3650 50  0001 C CNN
+	1    5300 3650
 	0    -1   1    0
 $EndComp

Commit message: cleaned up libs
Parts:
- U8: symbol otter:AP3019A -> OtterCastAmp-rescue:AP3019A-otter
Changed lines of the file:
@@
 LEDK
 $Comp
-L otter:AP3019A U8
+L OtterCastAmp-rescue:AP3019A-otter U8
 U 1 1 60C69466
 P 3550 2350

Commit message: V1.2 production release
Parts:
- removed JP10, JP9: JMP, Jumper:SolderJumper-2_P1.3mm_Bridged_Pad1.0x1.5mm, symbol Device:Jumper_NC_Small
- added R86, R87, R88: 0R, otter:R_0402, symbol Device:R_Small
- added TP1, TP2, TP3, TP4, TP5, TP6, TP7, TP8: TestPoint, TestPoint:TestPoint_Pad_1.0x1.0mm, symbol Connector:TestPoint
Connections:
- net B1: now also TP4.1
- net I2C0_INT: now also R88.2
- net I2C0_SCL: now also R86.2
- net I2C0_SDA: now also R87.2
- net LCD_DCLK: now also TP6.1
- net LCD_ENAB: now also TP5.1
- net LCD_HSYNC: now also TP7.1
- net LCD_VSYNC: now also TP8.1
- net LCD_SCL: now reaches J10.6 (Pin_6)
- net LCD_SCL: now also R86.1, TP2.1
- net LCD_CS: now reaches J10.7 (Pin_7)
- net LCD_CS: now also R88.1, TP3.1
- net LCD_SDA: now reaches J10.5 (Pin_5)
- net LCD_SDA: now also R87.1, TP1.1
- no-connect marks 5 -> 4
Changed lines of the file:
@@
 $EndComp
 NoConn ~ 7550 1250
-$Comp
-L Device:Jumper_NC_Small JP9
-U 1 1 60C3AE8C
-P 7250 1450
-F 0 "JP9" H 7100 1500 50  0000 C CNN
-F 1 "JMP" H 7400 1500 50  0000 C CNN
-F 2 "Jumper:SolderJumper-2_P1.3mm_Bridged_Pad1.0x1.5mm" H 7250 1450 50  0001 C CNN
-F 3 "~" H 7250 1450 50  0001 C CNN
-	1    7250 1450
-	1    0    0    -1
-$EndComp
-Wire Wire Line
-	7350 1550 7550 1550
-Wire Wire Line
-	7550 1450 7350 1450
-NoConn ~ 7550 1350
-$Comp
-L otter:GND #PWR0236
-U 1 1 60C3E844
-P 7000 1450
-F 0 "#PWR0236" H 7000 1200 50  0001 C CNN
-F 1 "GND" V 7000 1300 50  0000 R CNN
-F 2 "" H 7000 1450 60  0000 C CNN
-F 3 "" H 7000 1450 60  0000 C CNN
-	1    7000 1450
-	0    1    1    0
-$EndComp
-$Comp
-L otter:GND #PWR0237
-U 1 1 60C3EB01
-P 7000 1550
-F 0 "#PWR0237" H 7000 1300 50  0001 C CNN
-F 1 "GND" V 7000 1400 50  0000 R CNN
-F 2 "" H 7000 1550 60  0000 C CNN
-F 3 "" H 7000 1550 60  0000 C CNN
-	1    7000 1550
-	0    1    1    0
-$EndComp
-Wire Wire Line
-	7000 1550 7150 1550
-Wire Wire Line
-	7150 1450 7000 1450
-$Comp
-L Device:Jumper_NC_Small JP10
-U 1 1 60C3C276
-P 7250 1550
-F 0 "JP10" H 7100 1600 50  0000 C CNN
-F 1 "JMP" H 7400 1600 50  0000 C CNN
-F 2 "Jumper:SolderJumper-2_P1.3mm_Bridged_Pad1.0x1.5mm" H 7250 1550 50  0001 C CNN
-F 3 "~" H 7250 1550 50  0001 C CNN
-	1    7250 1550
-	1    0    0    -1
-$EndComp
 Text GLabel 7550 1650 0    50   Input ~ 0
 LCD_RESET
@@
 	0    -1   1    0
 $EndComp
+Text GLabel 7550 1350 0    50   Input ~ 0
+LCD_SDA
+Text GLabel 7550 1450 0    50   Input ~ 0
+LCD_SCL
+Text GLabel 7550 1550 0    50   Input ~ 0
+LCD_CS
+Text GLabel 5850 2600 0    50   Input ~ 0
+I2C0_SCL
+Text GLabel 5850 2700 0    50   Input ~ 0
+I2C0_SDA
+Text GLabel 5850 2800 0    50   Input ~ 0
+I2C0_INT
+$Comp
+L Device:R_Small R?
+U 1 1 6076BFC5
+P 6100 2600
+AR Path="/6076BFC5" Ref="R?"  Part="1"
+AR Path="/6145FE90/6076BFC5" Ref="R86"  Part="1"
+F 0 "R86" V 6050 2450 50  0000 C CNN
+F 1 "0R" V 6050 2800 50  0000 C CNN
+F 2 "otter:R_0402" H 6100 2600 50  0001 C CNN
+F 3 "~" H 6100 2600 50  0001 C CNN
+	1    6100 2600
+	0    1    1    0
+$EndComp
+$Comp
+L Device:R_Small R?
+U 1 1 6076C28C
+P 6100 2700
+AR Path="/6076C28C" Ref="R?"  Part="1"
+AR Path="/6145FE90/6076C28C" Ref="R87"  Part="1"
+F 0 "R87" V 6050 2550 50  0000 C CNN
+F 1 "0R" V 6050 2900 50  0000 C CNN
+F 2 "otter:R_0402" H 6100 2700 50  0001 C CNN
+F 3 "~" H 6100 2700 50  0001 C CNN
+	1    6100 2700
+	0    1    1    0
+$EndComp
+$Comp
+L Device:R_Small R?
+U 1 1 6076C4B4
+P 6100 2800
+AR Path="/6076C4B4" Ref="R?"  Part="1"
+AR Path="/6145FE90/6076C4B4" Ref="R88"  Part="1"
+F 0 "R88" V 6050 2650 50  0000 C CNN
+F 1 "0R" V 6050 3000 50  0000 C CNN
+F 2 "otter:R_0402" H 6100 2800 50  0001 C CNN
+F 3 "~" H 6100 2800 50  0001 C CNN
+	1    6100 2800
+	0    1    1    0
+$EndComp
+Text GLabel 6400 2700 2    50   Input ~ 0
+LCD_SDA
+Text GLabel 6400 2600 2    50   Input ~ 0
+LCD_SCL
+Text GLabel 6400 2800 2    50   Input ~ 0
+LCD_CS
+Wire Wire Line
+	6400 2600 6200 2600
+Wire Wire Line
+	6200 2700 6400 2700
+Wire Wire Line
+	6400 2800 6200 2800
+Wire Wire Line
+	6000 2800 5850 2800
+Wire Wire Line
+	5850 2700 6000 2700
+Wire Wire Line
+	6000 2600 5850 2600
+$Comp
+L Connector:TestPoint TP8
+U 1 1 6077A974
+P 7900 3650
+F 0 "TP8" V 7900 3838 50  0000 L CNN
+F 1 "TestPoint" V 7945 3838 50  0001 L CNN
+F 2 "TestPoint:TestPoint_Pad_1.0x1.0mm" H 8100 3650 50  0001 C CNN
+F 3 "~" H 8100 3650 50  0001 C CNN
+	1    7900 3650
+	0    1    1    0
+$EndComp
+$Comp
+L Connector:TestPoint TP7
+U 1 1 6077E3F5
+P 7900 3550
+F 0 "TP7" V 7900 3738 50  0000 L CNN
+F 1 "TestPoint" V 7945 3738 50  0001 L CNN
+F 2 "TestPoint:TestPoint_Pad_1.0x1.0mm" H 8100 3550 50  0001 C CNN
+F 3 "~" H 8100 3550 50  0001 C CNN
+	1    7900 3550
+	0    1    1    0
+$EndComp
+$Comp
+L Connector:TestPoint TP6
+U 1 1 6077E582
+P 7900 3450
+F 0 "TP6" V 7900 3638 50  0000 L CNN
+F 1 "TestPoint" V 7945 3638 50  0001 L CNN
+F 2 "TestPoint:TestPoint_Pad_1.0x1.0mm" H 8100 3450 50  0001 C CNN
+F 3 "~" H 8100 3450 50  0001 C CNN
+	1    7900 3450
+	0    1    1    0
+$EndComp
+$Comp
+L Connector:TestPoint TP5
+U 1 1 6077E815
+P 7900 3350
+F 0 "TP5" V 7900 3538 50  0000 L CNN
+F 1 "TestPoint" V 7945 3538 50  0001 L CNN
+F 2 "TestPoint:TestPoint_Pad_1.0x1.0mm" H 8100 3350 50  0001 C CNN
+F 3 "~" H 8100 3350 50  0001 C CNN
+	1    7900 3350
+	0    1    1    0
+$EndComp
+$Comp
+L Connector:TestPoint TP4
+U 1 1 6077EF76
+P 7900 3250
+F 0 "TP4" V 7900 3438 50  0000 L CNN
+F 1 "TestPoint" V 7945 3438 50  0001 L CNN
+F 2 "TestPoint:TestPoint_Pad_1.0x1.0mm" H 8100 3250 50  0001 C CNN
+F 3 "~" H 8100 3250 50  0001 C CNN
+	1    7900 3250
+	0    1    1    0
+$EndComp
+Wire Wire Line
+	7900 3250 7550 3250
+Wire Wire Line
+	7550 3350 7900 3350
+Wire Wire Line
+	7900 3450 7550 3450
+Wire Wire Line
+	7550 3550 7900 3550
+Wire Wire Line
+	7900 3650 7550 3650
+$Comp
+L Connector:TestPoint TP3
+U 1 1 6078578F
+P 7850 1550
+F 0 "TP3" V 7850 1738 50  0000 L CNN
+F 1 "TestPoint" V 7895 1738 50  0001 L CNN
+F 2 "TestPoint:TestPoint_Pad_1.0x1.0mm" H 8050 1550 50  0001 C CNN
+F 3 "~" H 8050 1550 50  0001 C CNN
+	1    7850 1550
+	0    1    1    0
+$EndComp
+$Comp
+L Connector:TestPoint TP2
+U 1 1 60785795
+P 7850 1450
+F 0 "TP2" V 7850 1638 50  0000 L CNN
+F 1 "TestPoint" V 7895 1638 50  0001 L CNN
+F 2 "TestPoint:TestPoint_Pad_1.0x1.0mm" H 8050 1450 50  0001 C CNN
+F 3 "~" H 8050 1450 50  0001 C CNN
+	1    7850 1450
+	0    1    1    0
+$EndComp
+$Comp
+L Connector:TestPoint TP1
+U 1 1 6078579B
+P 7850 1350
+F 0 "TP1" V 7850 1538 50  0000 L CNN
+F 1 "TestPoint" V 7895 1538 50  0001 L CNN
+F 2 "TestPoint:TestPoint_Pad_1.0x1.0mm" H 8050 1350 50  0001 C CNN
+F 3 "~" H 8050 1350 50  0001 C CNN
+	1    7850 1350
+	0    1    1    0
+$EndComp
+Wire Wire Line
+	7850 1350 7550 1350
+Wire Wire Line
+	7550 1450 7850 1450
+Wire Wire Line
+	7850 1550 7550 1550
 $EndSCHEMATC
