File: front/back.kicad_pcb (KiCad board)
At the start: 2 copper layers, 100 x 43 mm, 4 parts

Commit message: V1.2 production release
Other:
- board text added: "Hardware: @JanHenrikH, @FauthNiklas 2021 Software: @Manawyrm, @Toble_Miner Rev 1.2"
- board text removed: "Hardware: @JanHenrikH, @FauthNiklas 2021 Software: @Manawyrm, @Toble_Miner Rev 1.0"
Changed lines of the file:
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@@
     (effects (font (size 3 3) (thickness 0.4)) (justify left))
   )
-  (gr_text "Hardware: @JanHenrikH, @FauthNiklas      2021\nSoftware: @Manawyrm, @Toble_Miner     Rev 1.0" (at 107.9 96.75) (layer F.SilkS)
+  (gr_text "Hardware: @JanHenrikH, @FauthNiklas      2021\nSoftware: @Manawyrm, @Toble_Miner     Rev 1.2" (at 107.9 96.75) (layer F.SilkS)
     (effects (font (size 1 1) (thickness 0.18)) (justify left))
   )
